File: Receiver/AMP/rx_amp.kicad_pcb (KiCad board)
At the start: 2 copper layers, 30 x 30 mm, 13 parts, among them IC1 BGA616H6327XTSA1, J1 Signal_In, J2 Signal_Out, J3 Screw_Terminal_01x02

Commit message: Vendor project libraries; clean ERC/DRC on all boards
- Copy embedded footprints and symbols into each project's local library
  and repoint FPIDs / lib_ids so every project is self-contained
- Add sym-lib-table for tx_amplifier and preenfasis
- Sync footprint fields with the schematic (parity) and mark LMH34400 JP1 DNP
- Remove dangling copper arc and silkscreen overlap in LTC6268-10
- Fix LED ERC metadata errors
- All 8 boards: ERC and DRC clean (0 errors, 0 warnings)
Parts:
- C1, C2, C3: footprint Capacitor_SMD:C_0402_1005Metric_Pad0.74x0.62mm_HandSolder -> rx_amp:C_0402_1005Metric_Pad0.74x0.62mm_HandSolder
- H1, H3: footprint MountingHole:MountingHole_3.2mm_M3_DIN965 -> rx_amp:MountingHole_3.2mm_M3_DIN965
- J1, J2: footprint Connector_Coaxial:SMA_Samtec_SMA-J-P-X-ST-EM1_EdgeMount -> rx_amp:SMA_Samtec_SMA-J-P-X-ST-EM1_EdgeMount
- J3: footprint TerminalBlock_RND:TerminalBlock_RND_205-00001_1x02_P5.00mm_Horizontal -> rx_amp:TerminalBlock_RND_205-00001_1x02_P5.00mm_Horizontal
- L1, L2, R1: footprint Inductor_SMD:L_0603_1608Metric_Pad1.05x0.95mm_HandSolder -> rx_amp:L_0603_1608Metric_Pad1.05x0.95mm_HandSolder
- L3: value Ferrite Beads 220 OHM -> Ferrite Beads 220 OHM; footprint Inductor_SMD:L_0603_1608Metric_Pad1.05x0.95mm_HandSolder -> rx_amp:L_0603_1608Metric_Pad1.05x0.95mm_HandSolder
Changed lines of the file:
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@@
 	(net 8 "Net-(J3-Pin_2)")
 	(net 9 "Net-(C3-Pad1)")
-	(footprint "Inductor_SMD:L_0603_1608Metric_Pad1.05x0.95mm_HandSolder"
+	(footprint "rx_amp:L_0603_1608Metric_Pad1.05x0.95mm_HandSolder"
 		(layer "F.Cu")
 		(at 128.5 93.9)
@@
 			)
 		)
-		(property "Footprint" "Inductor_SMD:L_0603_1608Metric_Pad1.05x0.95mm_HandSolder"
+		(property "Footprint" "rx_amp:L_0603_1608Metric_Pad1.05x0.95mm_HandSolder"
 			(at 0 0 0)
 			(unlocked yes)
@@
 			)
 		)
-		(property "Description" "SMD WRIS-RSKS 15 Ohms 1 % 0.1 W 0603 "
+		(property "Description" "SMD WRIS-RSKS 15 Ohms 1 % 0.1 W 0603"
 			(at 0 0 0)
 			(unlocked yes)
@@
 		)
 	)
-	(footprint "MountingHole:MountingHole_3.2mm_M3_DIN965"
+	(footprint "rx_amp:MountingHole_3.2mm_M3_DIN965"
 		(layer "F.Cu")
 		(at 136 94)
@@
 			)
 		)
-		(property "Footprint" "MountingHole:MountingHole_3.2mm_M3_DIN965"
+		(property "Footprint" "rx_amp:MountingHole_3.2mm_M3_DIN965"
 			(at 0 0 0)
 			(unlocked yes)
@@
 		)
 	)
-	(footprint "Inductor_SMD:L_0603_1608Metric_Pad1.05x0.95mm_HandSolder"
+	(footprint "rx_amp:L_0603_1608Metric_Pad1.05x0.95mm_HandSolder"
 		(layer "F.Cu")
 		(at 125 96)
@@
 			)
 		)
-		(property "Value" " Ferrite Beads 220 OHM "
+		(property "Value" "Ferrite Beads 220 OHM"
 			(at 0 1.43 0)
 			(layer "F.Fab")
@@
 			)
 		)
-		(property "Footprint" "Inductor_SMD:L_0603_1608Metric_Pad1.05x0.95mm_HandSolder"
+		(property "Footprint" "rx_amp:L_0603_1608Metric_Pad1.05x0.95mm_HandSolder"
 			(at 0 0 0)
 			(unlocked yes)
@@
 			)
 		)
-		(property "Description" " Ferrite Beads 220 OHM 25% Alternate Sizing Guide Below "
+		(property "Description" "Ferrite Beads 220 OHM 25% Alternate Sizing Guide Below"
 			(at 0 0 0)
 			(unlocked yes)
@@
 		)
 	)
-	(footprint "Capacitor_SMD:C_0402_1005Metric_Pad0.74x0.62mm_HandSolder"
+	(footprint "rx_amp:C_0402_1005Metric_Pad0.74x0.62mm_HandSolder"
 		(layer "F.Cu")
 		(at 126 100 -90)
@@
 			)
 		)
-		(property "Footprint" "Capacitor_SMD:C_0402_1005Metric_Pad0.74x0.62mm_HandSolder"
+		(property "Footprint" "rx_amp:C_0402_1005Metric_Pad0.74x0.62mm_HandSolder"
 			(at 0 0 -90)
 			(unlocked yes)
@@
 			)
 		)
-		(property "Description" "16V 10nF 10% Tin Plated Chip "
+		(property "Description" "16V 10nF 10% Tin Plated Chip"
 			(at 0 0 -90)
 			(unlocked yes)
@@
 		)
 	)
-	(footprint "Capacitor_SMD:C_0402_1005Metric_Pad0.74x0.62mm_HandSolder"
+	(footprint "rx_amp:C_0402_1005Metric_Pad0.74x0.62mm_HandSolder"
 		(layer "F.Cu")
 		(at 133 107)
@@
 			)
 		)
-		(property "Footprint" "Capacitor_SMD:C_0402_1005Metric_Pad0.74x0.62mm_HandSolder"
+		(property "Footprint" "rx_amp:C_0402_1005Metric_Pad0.74x0.62mm_HandSolder"
 			(at 0 0 0)
 			(unlocked yes)
@@
 			)
 		)
-		(property "Description" "16V 10nF 10% Tin Plated Chip "
+		(property "Description" "16V 10nF 10% Tin Plated Chip"
 			(at 0 0 0)
 			(unlocked yes)
@@
 		)
 	)
-	(footprint "Connector_Coaxial:SMA_Samtec_SMA-J-P-X-ST-EM1_EdgeMount"
+	(footprint "rx_amp:SMA_Samtec_SMA-J-P-X-ST-EM1_EdgeMount"
 		(layer "F.Cu")
 		(at 137.5 107 90)
@@
 			)
 		)
-		(property "Footprint" "Connector_Coaxial:SMA_Samtec_SMA-J-P-X-ST-EM1_EdgeMount"
+		(property "Footprint" "rx_amp:SMA_Samtec_SMA-J-P-X-ST-EM1_EdgeMount"
 			(at 0 0 90)
 			(unlocked yes)
@@
 			)
 		)
-		(property "Datasheet" " ~"
+		(property "Datasheet" "~"
 			(at 0 0 90)
 			(unlocked yes)
@@
 		)
 	)
-	(footprint "Connector_Coaxial:SMA_Samtec_SMA-J-P-X-ST-EM1_EdgeMount"
+	(footprint "rx_amp:SMA_Samtec_SMA-J-P-X-ST-EM1_EdgeMount"
 		(layer "F.Cu")
 		(at 112.5 111 -90)
@@
 			)
 		)
-		(property "Footprint" "Connector_Coaxial:SMA_Samtec_SMA-J-P-X-ST-EM1_EdgeMount"
+		(property "Footprint" "rx_amp:SMA_Samtec_SMA-J-P-X-ST-EM1_EdgeMount"
 			(at 0 0 -90)
 			(unlocked yes)
@@
 			)
 		)
-		(property "Datasheet" " ~"
+		(property "Datasheet" "~"
 			(at 0 0 -90)
 			(unlocked yes)
@@
 		)
 	)
-	(footprint "Inductor_SMD:L_0603_1608Metric_Pad1.05x0.95mm_HandSolder"
+	(footprint "rx_amp:L_0603_1608Metric_Pad1.05x0.95mm_HandSolder"
 		(layer "F.Cu")
 		(at 131 103 -90)
@@
 			)
 		)
-		(property "Footprint" "Inductor_SMD:L_0603_1608Metric_Pad1.05x0.95mm_HandSolder"
+		(property "Footprint" "rx_amp:L_0603_1608Metric_Pad1.05x0.95mm_HandSolder"
 			(at 0 0 -90)
 			(unlocked yes)
@@
 		)
 	)
-	(footprint "Inductor_SMD:L_0603_1608Metric_Pad1.05x0.95mm_HandSolder"
+	(footprint "rx_amp:L_0603_1608Metric_Pad1.05x0.95mm_HandSolder"
 		(layer "F.Cu")
 		(at 131 98 -90)
@@
 			)
 		)
-		(property "Footprint" "Inductor_SMD:L_0603_1608Metric_Pad1.05x0.95mm_HandSolder"
+		(property "Footprint" "rx_amp:L_0603_1608Metric_Pad1.05x0.95mm_HandSolder"
 			(at 0 0 -90)
 			(unlocked yes)
@@
 		)
 	)
-	(footprint "Capacitor_SMD:C_0402_1005Metric_Pad0.74x0.62mm_HandSolder"
+	(footprint "rx_amp:C_0402_1005Metric_Pad0.74x0.62mm_HandSolder"
 		(layer "F.Cu")
 		(at 118 111)
@@
 			)
 		)
-		(property "Footprint" "Capacitor_SMD:C_0402_1005Metric_Pad0.74x0.62mm_HandSolder"
+		(property "Footprint" "rx_amp:C_0402_1005Metric_Pad0.74x0.62mm_HandSolder"
 			(at 0 0 0)
 			(unlocked yes)
@@
 			)
 		)
-		(property "Description" "16V 10nF 10% Tin Plated Chip "
+		(property "Description" "16V 10nF 10% Tin Plated Chip"
 			(at 0 0 0)
 			(unlocked yes)
@@
 		)
 	)
-	(footprint "TerminalBlock_RND:TerminalBlock_RND_205-00001_1x02_P5.00mm_Horizontal"
+	(footprint "rx_amp:TerminalBlock_RND_205-00001_1x02_P5.00mm_Horizontal"
 		(layer "F.Cu")
 		(at 115 96.5)
@@
 			)
 		)
-		(property "Footprint" "TerminalBlock_RND:TerminalBlock_RND_205-00001_1x02_P5.00mm_Horizontal"
+		(property "Footprint" "rx_amp:TerminalBlock_RND_205-00001_1x02_P5.00mm_Horizontal"
 			(at 0 0 0)
 			(unlocked yes)
@@
 		)
 	)
-	(footprint "MountingHole:MountingHole_3.2mm_M3_DIN965"
+	(footprint "rx_amp:MountingHole_3.2mm_M3_DIN965"
 		(layer "F.Cu")
 		(at 136 116)
@@
 			)
 		)
-		(property "Footprint" "MountingHole:MountingHole_3.2mm_M3_DIN965"
+		(property "Footprint" "rx_amp:MountingHole_3.2mm_M3_DIN965"
 			(at 0 0 0)
 			(unlocked yes)
