File: Receiver/AMP/rx_amp.kicad_sch (KiCad schematic)
At the start: 13 parts, among them IC1 BGA616H6327XTSA1, J1 Signal_In, J2 Signal_Out, J3 Screw_Terminal_01x02

Commit message: Vendor project libraries; clean ERC/DRC on all boards
- Copy embedded footprints and symbols into each project's local library
  and repoint FPIDs / lib_ids so every project is self-contained
- Add sym-lib-table for tx_amplifier and preenfasis
- Sync footprint fields with the schematic (parity) and mark LMH34400 JP1 DNP
- Remove dangling copper arc and silkscreen overlap in LTC6268-10
- Fix LED ERC metadata errors
- All 8 boards: ERC and DRC clean (0 errors, 0 warnings)
Parts:
- C1, C2, C3: footprint Capacitor_SMD:C_0402_1005Metric_Pad0.74x0.62mm_HandSolder -> rx_amp:C_0402_1005Metric_Pad0.74x0.62mm_HandSolder; symbol Device:C_Small -> rx_amp:C_Small
- H1, H3: footprint MountingHole:MountingHole_3.2mm_M3_DIN965 -> rx_amp:MountingHole_3.2mm_M3_DIN965; symbol Mechanical:MountingHole -> rx_amp:MountingHole
- J1, J2: footprint Connector_Coaxial:SMA_Samtec_SMA-J-P-X-ST-EM1_EdgeMount -> rx_amp:SMA_Samtec_SMA-J-P-X-ST-EM1_EdgeMount; symbol Connector:Conn_Coaxial -> rx_amp:Conn_Coaxial
- J3: footprint TerminalBlock_RND:TerminalBlock_RND_205-00001_1x02_P5.00mm_Horizontal -> rx_amp:TerminalBlock_RND_205-00001_1x02_P5.00mm_Horizontal; symbol Connector:Screw_Terminal_01x02 -> rx_amp:Screw_Terminal_01x02
- L1, L2: footprint Inductor_SMD:L_0603_1608Metric_Pad1.05x0.95mm_HandSolder -> rx_amp:L_0603_1608Metric_Pad1.05x0.95mm_HandSolder; symbol Device:L_Small -> rx_amp:L_Small
- L3: footprint Inductor_SMD:L_0603_1608Metric_Pad1.05x0.95mm_HandSolder -> rx_amp:L_0603_1608Metric_Pad1.05x0.95mm_HandSolder; symbol Device:L_Ferrite_Small -> rx_amp:L_Ferrite_Small
- R1: footprint Inductor_SMD:L_0603_1608Metric_Pad1.05x0.95mm_HandSolder -> rx_amp:L_0603_1608Metric_Pad1.05x0.95mm_HandSolder; symbol Device:R_Small_US -> rx_amp:R_Small_US
Changed lines of the file:
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@@
 	)
 	(symbol
-		(lib_id "power:GND")
+		(lib_id "rx_amp:GND")
 		(at 137.16 104.14 0)
 		(unit 1)
@@
 	)
 	(symbol
-		(lib_id "Device:L_Small")
+		(lib_id "rx_amp:L_Small")
 		(at 177.8 76.2 0)
 		(unit 1)
@@
 			)
 		)
-		(property "Footprint" "Inductor_SMD:L_0603_1608Metric_Pad1.05x0.95mm_HandSolder"
+		(property "Footprint" "rx_amp:L_0603_1608Metric_Pad1.05x0.95mm_HandSolder"
 			(at 177.8 76.2 0)
 			(effects
@@
 	)
 	(symbol
-		(lib_id "power:GND")
+		(lib_id "rx_amp:GND")
 		(at 88.9 106.68 0)
 		(unit 1)
@@
 	)
 	(symbol
-		(lib_id "Device:C_Small")
+		(lib_id "rx_amp:C_Small")
 		(at 198.12 104.14 90)
 		(unit 1)
@@
 			)
 		)
-		(property "Footprint" "Capacitor_SMD:C_0402_1005Metric_Pad0.74x0.62mm_HandSolder"
+		(property "Footprint" "rx_amp:C_0402_1005Metric_Pad0.74x0.62mm_HandSolder"
 			(at 198.12 104.14 0)
 			(effects
@@
 	)
 	(symbol
-		(lib_id "Connector:Conn_Coaxial")
+		(lib_id "rx_amp:Conn_Coaxial")
 		(at 215.9 104.14 0)
 		(unit 1)
@@
 			)
 		)
-		(property "Footprint" "Connector_Coaxial:SMA_Samtec_SMA-J-P-X-ST-EM1_EdgeMount"
+		(property "Footprint" "rx_amp:SMA_Samtec_SMA-J-P-X-ST-EM1_EdgeMount"
 			(at 215.9 104.14 0)
 			(effects
@@
 	)
 	(symbol
-		(lib_id "power:GND")
+		(lib_id "rx_amp:GND")
 		(at 132.08 66.04 0)
 		(unit 1)
@@
 	)
 	(symbol
-		(lib_id "power:PWR_FLAG")
+		(lib_id "rx_amp:PWR_FLAG")
 		(at 137.16 50.8 0)
 		(unit 1)
@@
 	)
 	(symbol
-		(lib_id "Device:L_Ferrite_Small")
+		(lib_id "rx_amp:L_Ferrite_Small")
 		(at 154.94 50.8 90)
 		(unit 1)
@@
 			)
 		)
-		(property "Footprint" "Inductor_SMD:L_0603_1608Metric_Pad1.05x0.95mm_HandSolder"
+		(property "Footprint" "rx_amp:L_0603_1608Metric_Pad1.05x0.95mm_HandSolder"
 			(at 154.94 50.8 0)
 			(effects
@@
 	)
 	(symbol
-		(lib_id "power:GND")
+		(lib_id "rx_amp:GND")
 		(at 170.18 106.68 0)
 		(unit 1)
@@
 	)
 	(symbol
-		(lib_id "Device:R_Small_US")
+		(lib_id "rx_amp:R_Small_US")
 		(at 177.8 63.5 0)
 		(unit 1)
@@
 			)
 		)
-		(property "Footprint" "Inductor_SMD:L_0603_1608Metric_Pad1.05x0.95mm_HandSolder"
+		(property "Footprint" "rx_amp:L_0603_1608Metric_Pad1.05x0.95mm_HandSolder"
 			(at 177.8 63.5 0)
 			(effects
@@
 	)
 	(symbol
-		(lib_id "power:GND")
+		(lib_id "rx_amp:GND")
 		(at 215.9 111.76 0)
 		(unit 1)
@@
 	)
 	(symbol
-		(lib_id "Connector:Conn_Coaxial")
+		(lib_id "rx_amp:Conn_Coaxial")
 		(at 88.9 101.6 0)
 		(mirror y)
@@
 			)
 		)
-		(property "Footprint" "Connector_Coaxial:SMA_Samtec_SMA-J-P-X-ST-EM1_EdgeMount"
+		(property "Footprint" "rx_amp:SMA_Samtec_SMA-J-P-X-ST-EM1_EdgeMount"
 			(at 88.9 101.6 0)
 			(effects
@@
 	)
 	(symbol
-		(lib_id "power:GND")
+		(lib_id "rx_amp:GND")
 		(at 203.2 53.34 0)
 		(unit 1)
@@
 	)
 	(symbol
-		(lib_id "Connector:Screw_Terminal_01x02")
+		(lib_id "rx_amp:Screw_Terminal_01x02")
 		(at 127 53.34 180)
 		(unit 1)
@@
 			)
 		)
-		(property "Footprint" "TerminalBlock_RND:TerminalBlock_RND_205-00001_1x02_P5.00mm_Horizontal"
+		(property "Footprint" "rx_amp:TerminalBlock_RND_205-00001_1x02_P5.00mm_Horizontal"
 			(at 127 53.34 0)
 			(effects
@@
 	)
 	(symbol
-		(lib_id "Device:L_Small")
+		(lib_id "rx_amp:L_Small")
 		(at 177.8 88.9 0)
 		(unit 1)
@@
 			)
 		)
-		(property "Footprint" "Inductor_SMD:L_0603_1608Metric_Pad1.05x0.95mm_HandSolder"
+		(property "Footprint" "rx_amp:L_0603_1608Metric_Pad1.05x0.95mm_HandSolder"
 			(at 177.8 88.9 0)
 			(effects
@@
 	)
 	(symbol
-		(lib_id "Mechanical:MountingHole")
+		(lib_id "rx_amp:MountingHole")
 		(at 228.6 63.5 0)
 		(unit 1)
@@
 			)
 		)
-		(property "Footprint" "MountingHole:MountingHole_3.2mm_M3_DIN965"
+		(property "Footprint" "rx_amp:MountingHole_3.2mm_M3_DIN965"
 			(at 228.6 63.5 0)
 			(effects
@@
 	)
 	(symbol
-		(lib_id "Mechanical:MountingHole")
+		(lib_id "rx_amp:MountingHole")
 		(at 228.6 76.2 0)
 		(unit 1)
@@
 			)
 		)
-		(property "Footprint" "MountingHole:MountingHole_3.2mm_M3_DIN965"
+		(property "Footprint" "rx_amp:MountingHole_3.2mm_M3_DIN965"
 			(at 228.6 76.2 0)
 			(effects
@@
 	)
 	(symbol
-		(lib_id "Device:C_Small")
+		(lib_id "rx_amp:C_Small")
 		(at 193.04 50.8 90)
 		(unit 1)
@@
 			)
 		)
-		(property "Footprint" "Capacitor_SMD:C_0402_1005Metric_Pad0.74x0.62mm_HandSolder"
+		(property "Footprint" "rx_amp:C_0402_1005Metric_Pad0.74x0.62mm_HandSolder"
 			(at 193.04 50.8 0)
 			(effects
@@
 	)
 	(symbol
-		(lib_id "Device:C_Small")
+		(lib_id "rx_amp:C_Small")
 		(at 114.3 101.6 90)
 		(unit 1)
@@
 			)
 		)
-		(property "Footprint" "Capacitor_SMD:C_0402_1005Metric_Pad0.74x0.62mm_HandSolder"
+		(property "Footprint" "rx_amp:C_0402_1005Metric_Pad0.74x0.62mm_HandSolder"
 			(at 114.3 101.6 0)
 			(effects
@@
 	)
 	(symbol
-		(lib_id "power:PWR_FLAG")
+		(lib_id "rx_amp:PWR_FLAG")
 		(at 132.08 63.5 270)
 		(unit 1)
