File: Receiver/PD/PD.kicad_pcb (KiCad board)
At the start: 2 copper layers, 32 x 34 mm, 9 parts, among them J2 RFPC-SMA28-F, J3 RFPC-SMA28-F, J4 RFPC-SMA28-F, J5 Screw_Terminal_01x02

Commit message: Vendor project libraries; clean ERC/DRC on all boards
- Copy embedded footprints and symbols into each project's local library
  and repoint FPIDs / lib_ids so every project is self-contained
- Add sym-lib-table for tx_amplifier and preenfasis
- Sync footprint fields with the schematic (parity) and mark LMH34400 JP1 DNP
- Remove dangling copper arc and silkscreen overlap in LTC6268-10
- Fix LED ERC metadata errors
- All 8 boards: ERC and DRC clean (0 errors, 0 warnings)
Parts:
- C1: footprint Capacitor_SMD:C_0603_1608Metric_Pad1.08x0.95mm_HandSolder -> Lumicom_Photodiode:C_0603_1608Metric_Pad1.08x0.95mm_HandSolder
- D1: footprint Package_TO_SOT_THT:TO-18-3 -> Lumicom_Photodiode:TO-18-3
- D3: footprint LED_THT:LED_D5.0mm_IRGrey -> Lumicom_Photodiode:LED_D5.0mm_IRGrey
- J5: footprint TerminalBlock:TerminalBlock_bornier-2_P5.08mm -> Lumicom_Photodiode:TerminalBlock_bornier-2_P5.08mm
- L1: footprint Inductor_SMD:L_0603_1608Metric_Pad1.05x0.95mm_HandSolder -> Lumicom_Photodiode:L_0603_1608Metric_Pad1.05x0.95mm_HandSolder
Changed lines of the file:
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@@
 	(net 5 "Net-(D3-A)")
 	(net 6 "Net-(J5-Pin_2)")
-	(footprint "Package_TO_SOT_THT:TO-18-3"
+	(footprint "Lumicom_Photodiode:TO-18-3"
 		(layer "F.Cu")
 		(at 114.414724 67.184724)
@@
 			)
 		)
-		(property "Footprint" "Package_TO_SOT_THT:TO-18-3"
+		(property "Footprint" "Lumicom_Photodiode:TO-18-3"
 			(at 0 0 0)
 			(layer "F.Fab")
@@
 		)
 	)
-	(footprint "LED_THT:LED_D5.0mm_IRGrey"
+	(footprint "Lumicom_Photodiode:LED_D5.0mm_IRGrey"
 		(layer "F.Cu")
 		(at 114.725 88)
@@
 			)
 		)
-		(property "Footprint" "LED_THT:LED_D5.0mm_IRGrey"
+		(property "Footprint" "Lumicom_Photodiode:LED_D5.0mm_IRGrey"
 			(at 0 0 0)
 			(layer "F.Fab")
@@
 		)
 	)
-	(footprint "Inductor_SMD:L_0603_1608Metric_Pad1.05x0.95mm_HandSolder"
+	(footprint "Lumicom_Photodiode:L_0603_1608Metric_Pad1.05x0.95mm_HandSolder"
 		(layer "F.Cu")
 		(at 106 77.5 -90)
@@
 			)
 		)
-		(property "Footprint" "Inductor_SMD:L_0603_1608Metric_Pad1.05x0.95mm_HandSolder"
+		(property "Footprint" "Lumicom_Photodiode:L_0603_1608Metric_Pad1.05x0.95mm_HandSolder"
 			(at 0 0 -90)
 			(unlocked yes)
@@
 		)
 	)
-	(footprint "Capacitor_SMD:C_0603_1608Metric_Pad1.08x0.95mm_HandSolder"
+	(footprint "Lumicom_Photodiode:C_0603_1608Metric_Pad1.08x0.95mm_HandSolder"
 		(layer "F.Cu")
 		(at 106 84 -90)
@@
 			)
 		)
-		(property "Footprint" "Capacitor_SMD:C_0603_1608Metric_Pad1.08x0.95mm_HandSolder"
+		(property "Footprint" "Lumicom_Photodiode:C_0603_1608Metric_Pad1.08x0.95mm_HandSolder"
 			(at 0 0 -90)
 			(unlocked yes)
@@
 		)
 	)
-	(footprint "TerminalBlock:TerminalBlock_bornier-2_P5.08mm"
+	(footprint "Lumicom_Photodiode:TerminalBlock_bornier-2_P5.08mm"
 		(layer "B.Cu")
 		(at 106 66 -90)
@@
 			)
 		)
-		(property "Footprint" "TerminalBlock:TerminalBlock_bornier-2_P5.08mm"
+		(property "Footprint" "Lumicom_Photodiode:TerminalBlock_bornier-2_P5.08mm"
 			(at 0 0 90)
 			(unlocked yes)
@@
 			)
 		)
-		(property "Datasheet" " ~"
+		(property "Datasheet" "~"
 			(at 0 0 0)
 			(unlocked yes)
@@
 			)
 		)
-		(property "Datasheet" " ~"
+		(property "Datasheet" "~"
 			(at 0 0 0)
 			(unlocked yes)
@@
 			)
 		)
-		(property "Datasheet" " ~"
+		(property "Datasheet" "~"
 			(at 0 0 0)
 			(unlocked yes)
