File: Receiver/PD/PD.kicad_sch (KiCad schematic)
At the start: 9 parts, among them J2 RFPC-SMA28-F, J3 RFPC-SMA28-F, J4 RFPC-SMA28-F, J5 Screw_Terminal_01x02

Commit message: Vendor project libraries; clean ERC/DRC on all boards
- Copy embedded footprints and symbols into each project's local library
  and repoint FPIDs / lib_ids so every project is self-contained
- Add sym-lib-table for tx_amplifier and preenfasis
- Sync footprint fields with the schematic (parity) and mark LMH34400 JP1 DNP
- Remove dangling copper arc and silkscreen overlap in LTC6268-10
- Fix LED ERC metadata errors
- All 8 boards: ERC and DRC clean (0 errors, 0 warnings)
Parts:
- C1: footprint Capacitor_SMD:C_0603_1608Metric_Pad1.08x0.95mm_HandSolder -> Lumicom_Photodiode:C_0603_1608Metric_Pad1.08x0.95mm_HandSolder; symbol Device:C_Small -> Lumicom_Photodiode:C_Small
- D1: footprint Package_TO_SOT_THT:TO-18-3 -> Lumicom_Photodiode:TO-18-3; symbol Sensor_Optical:S5971 -> Lumicom_Photodiode:S5971
- D3: footprint LED_THT:LED_D5.0mm_IRGrey -> Lumicom_Photodiode:LED_D5.0mm_IRGrey; symbol Sensor_Optical:SFH203 -> Lumicom_Photodiode:SFH203
- J2, J3, J4: symbol Connector:Conn_Coaxial -> Lumicom_Photodiode:Conn_Coaxial
- J5: footprint TerminalBlock:TerminalBlock_bornier-2_P5.08mm -> Lumicom_Photodiode:TerminalBlock_bornier-2_P5.08mm; symbol Connector:Screw_Terminal_01x02 -> Lumicom_Photodiode:Screw_Terminal_01x02
- L1: footprint Inductor_SMD:L_0603_1608Metric_Pad1.05x0.95mm_HandSolder -> Lumicom_Photodiode:L_0603_1608Metric_Pad1.05x0.95mm_HandSolder; symbol Device:L_Ferrite_Small -> Lumicom_Photodiode:L_Ferrite_Small
Changed lines of the file:
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@@
 	)
 	(symbol
-		(lib_id "Sensor_Optical:SFH203")
+		(lib_id "Lumicom_Photodiode:SFH203")
 		(at 142.24 118.11 0)
 		(unit 1)
@@
 			)
 		)
-		(property "Footprint" "LED_THT:LED_D5.0mm_IRGrey"
+		(property "Footprint" "Lumicom_Photodiode:LED_D5.0mm_IRGrey"
 			(at 142.24 113.665 0)
 			(effects
@@
 	)
 	(symbol
-		(lib_id "Connector:Conn_Coaxial")
+		(lib_id "Lumicom_Photodiode:Conn_Coaxial")
 		(at 198.12 71.12 0)
 		(unit 1)
@@
 	)
 	(symbol
-		(lib_id "power:GND")
+		(lib_id "Lumicom_Photodiode:GND")
 		(at 198.12 106.68 0)
 		(unit 1)
@@
 	)
 	(symbol
-		(lib_id "power:GND")
+		(lib_id "Lumicom_Photodiode:GND")
 		(at 69.85 76.2 0)
 		(unit 1)
@@
 	)
 	(symbol
-		(lib_id "power:GND")
+		(lib_id "Lumicom_Photodiode:GND")
 		(at 99.06 83.82 0)
 		(unit 1)
@@
 	)
 	(symbol
-		(lib_id "Connector:Conn_Coaxial")
+		(lib_id "Lumicom_Photodiode:Conn_Coaxial")
 		(at 198.12 99.06 0)
 		(unit 1)
@@
 	)
 	(symbol
-		(lib_id "power:GND")
+		(lib_id "Lumicom_Photodiode:GND")
 		(at 142.24 80.01 0)
 		(unit 1)
@@
 	)
 	(symbol
-		(lib_id "Connector:Conn_Coaxial")
+		(lib_id "Lumicom_Photodiode:Conn_Coaxial")
 		(at 198.12 118.11 0)
 		(unit 1)
@@
 	)
 	(symbol
-		(lib_id "Device:C_Small")
+		(lib_id "Lumicom_Photodiode:C_Small")
 		(at 99.06 78.74 0)
 		(unit 1)
@@
 			)
 		)
-		(property "Footprint" "Capacitor_SMD:C_0603_1608Metric_Pad1.08x0.95mm_HandSolder"
+		(property "Footprint" "Lumicom_Photodiode:C_0603_1608Metric_Pad1.08x0.95mm_HandSolder"
 			(at 99.06 78.74 0)
 			(effects
@@
 	)
 	(symbol
-		(lib_id "Device:L_Ferrite_Small")
+		(lib_id "Lumicom_Photodiode:L_Ferrite_Small")
 		(at 88.9 71.12 90)
 		(unit 1)
@@
 			)
 		)
-		(property "Footprint" "Inductor_SMD:L_0603_1608Metric_Pad1.05x0.95mm_HandSolder"
+		(property "Footprint" "Lumicom_Photodiode:L_0603_1608Metric_Pad1.05x0.95mm_HandSolder"
 			(at 88.9 71.12 0)
 			(effects
@@
 	)
 	(symbol
-		(lib_id "power:GND")
+		(lib_id "Lumicom_Photodiode:GND")
 		(at 198.12 125.73 0)
 		(unit 1)
@@
 	)
 	(symbol
-		(lib_id "power:PWR_FLAG")
+		(lib_id "Lumicom_Photodiode:PWR_FLAG")
 		(at 69.85 74.93 270)
 		(unit 1)
@@
 	)
 	(symbol
-		(lib_id "Sensor_Optical:S5971")
+		(lib_id "Lumicom_Photodiode:S5971")
 		(at 142.24 71.12 0)
 		(unit 1)
@@
 			)
 		)
-		(property "Footprint" "Package_TO_SOT_THT:TO-18-3"
+		(property "Footprint" "Lumicom_Photodiode:TO-18-3"
 			(at 142.24 62.23 0)
 			(effects
@@
 	)
 	(symbol
-		(lib_id "power:GND")
+		(lib_id "Lumicom_Photodiode:GND")
 		(at 198.12 78.74 0)
 		(unit 1)
@@
 	)
 	(symbol
-		(lib_id "Connector:Screw_Terminal_01x02")
+		(lib_id "Lumicom_Photodiode:Screw_Terminal_01x02")
 		(at 63.5 73.66 180)
 		(unit 1)
@@
 			)
 		)
-		(property "Footprint" "TerminalBlock:TerminalBlock_bornier-2_P5.08mm"
+		(property "Footprint" "Lumicom_Photodiode:TerminalBlock_bornier-2_P5.08mm"
 			(at 63.5 73.66 0)
 			(effects
