File: Receiver/TIA/LMH34400/LMH34400.kicad_pcb (KiCad board)
At the start: 4 copper layers, 34 x 40 mm, 24 parts, among them J1 TEST, J2 PD IN, J3 Vout, J4 N_EN, J5 N_ALC, J6 OUT, U1 LMH34400

Commit message: Vendor project libraries; clean ERC/DRC on all boards
- Copy embedded footprints and symbols into each project's local library
  and repoint FPIDs / lib_ids so every project is self-contained
- Add sym-lib-table for tx_amplifier and preenfasis
- Sync footprint fields with the schematic (parity) and mark LMH34400 JP1 DNP
- Remove dangling copper arc and silkscreen overlap in LTC6268-10
- Fix LED ERC metadata errors
- All 8 boards: ERC and DRC clean (0 errors, 0 warnings)
Parts:
- C1, C2, C6: footprint Capacitor_SMD:C_0402_1005Metric_Pad0.74x0.62mm_HandSolder -> LumiCom_TIA:C_0402_1005Metric_Pad0.74x0.62mm_HandSolder
- C3, C4, C5: footprint Capacitor_SMD:C_0603_1608Metric_Pad1.08x0.95mm_HandSolder -> LumiCom_TIA:C_0603_1608Metric_Pad1.08x0.95mm_HandSolder
- D1: footprint LED_SMD:LED_0603_1608Metric -> LumiCom_TIA:LED_0603_1608Metric
- H1, H2, H3: footprint MountingHole:MountingHole_3.2mm_M3_DIN965 -> LumiCom_TIA:MountingHole_3.2mm_M3_DIN965
- J1, J2, J6: footprint Connector_Coaxial:SMA_Samtec_SMA-J-P-X-ST-EM1_EdgeMount -> LumiCom_TIA:SMA_Samtec_SMA-J-P-X-ST-EM1_EdgeMount
- J3: footprint TerminalBlock_Phoenix:TerminalBlock_Phoenix_MKDS-1,5-2_1x02_P5.00mm_Horizontal -> LumiCom_TIA:TerminalBlock_Phoenix_MKDS-1,5-2_1x02_P5.00mm_Horizontal
- J4, J5: footprint Connector_PinHeader_2.54mm:PinHeader_1x03_P2.54mm_Vertical -> LumiCom_TIA:PinHeader_1x03_P2.54mm_Vertical
- JP1, R1, R2, R3, R4, R5: footprint Resistor_SMD:R_0603_1608Metric_Pad0.98x0.95mm_HandSolder -> LumiCom_TIA:R_0603_1608Metric_Pad0.98x0.95mm_HandSolder
- L1: value Ferrite Beads 220 OHM -> Ferrite Beads 220 OHM; footprint Inductor_SMD:L_0603_1608Metric_Pad1.05x0.95mm_HandSolder -> LumiCom_TIA:L_0603_1608Metric_Pad1.05x0.95mm_HandSolder
