File: Receiver/TIA/LMH34400/LMH34400.kicad_sch (KiCad schematic)
At the start: 24 parts, among them J1 TEST, J2 PD IN, J3 Vout, J4 N_EN, J5 N_ALC, J6 OUT, U1 LMH34400

Commit message: Vendor project libraries; clean ERC/DRC on all boards
- Copy embedded footprints and symbols into each project's local library
  and repoint FPIDs / lib_ids so every project is self-contained
- Add sym-lib-table for tx_amplifier and preenfasis
- Sync footprint fields with the schematic (parity) and mark LMH34400 JP1 DNP
- Remove dangling copper arc and silkscreen overlap in LTC6268-10
- Fix LED ERC metadata errors
- All 8 boards: ERC and DRC clean (0 errors, 0 warnings)
Parts:
- C1, C2, C6: footprint Capacitor_SMD:C_0402_1005Metric_Pad0.74x0.62mm_HandSolder -> LumiCom_TIA:C_0402_1005Metric_Pad0.74x0.62mm_HandSolder; symbol Device:C_Small -> LumiCom_TIA:C_Small
- C3, C4, C5: footprint Capacitor_SMD:C_0603_1608Metric_Pad1.08x0.95mm_HandSolder -> LumiCom_TIA:C_0603_1608Metric_Pad1.08x0.95mm_HandSolder; symbol Device:C_Small -> LumiCom_TIA:C_Small
- D1: footprint LED_SMD:LED_0603_1608Metric -> LumiCom_TIA:LED_0603_1608Metric; symbol Device:LED -> LumiCom_TIA:LED
- H1, H2, H3: footprint MountingHole:MountingHole_3.2mm_M3_DIN965 -> LumiCom_TIA:MountingHole_3.2mm_M3_DIN965; symbol Mechanical:MountingHole -> LumiCom_TIA:MountingHole
- J1, J2, J6: footprint Connector_Coaxial:SMA_Samtec_SMA-J-P-X-ST-EM1_EdgeMount -> LumiCom_TIA:SMA_Samtec_SMA-J-P-X-ST-EM1_EdgeMount; symbol Connector:Conn_Coaxial -> LumiCom_TIA:Conn_Coaxial
- J3: footprint TerminalBlock_Phoenix:TerminalBlock_Phoenix_MKDS-1,5-2_1x02_P5.00mm_Horizontal -> LumiCom_TIA:TerminalBlock_Phoenix_MKDS-1,5-2_1x02_P5.00mm_Horizontal; symbol Connector:Screw_Terminal_01x02 -> LumiCom_TIA:Screw_Terminal_01x02
- J4, J5: footprint Connector_PinHeader_2.54mm:PinHeader_1x03_P2.54mm_Vertical -> LumiCom_TIA:PinHeader_1x03_P2.54mm_Vertical; symbol Connector_Generic:Conn_01x03 -> LumiCom_TIA:Conn_01x03
- JP1: footprint Resistor_SMD:R_0603_1608Metric_Pad0.98x0.95mm_HandSolder -> LumiCom_TIA:R_0603_1608Metric_Pad0.98x0.95mm_HandSolder; symbol Jumper:SolderJumper_2_Open -> LumiCom_TIA:SolderJumper_2_Open; now not fitted
- L1: footprint Inductor_SMD:L_0603_1608Metric_Pad1.05x0.95mm_HandSolder -> LumiCom_TIA:L_0603_1608Metric_Pad1.05x0.95mm_HandSolder; symbol Device:L_Ferrite_Small -> LumiCom_TIA:L_Ferrite_Small
- R1, R2, R3, R4, R5: footprint Resistor_SMD:R_0603_1608Metric_Pad0.98x0.95mm_HandSolder -> LumiCom_TIA:R_0603_1608Metric_Pad0.98x0.95mm_HandSolder; symbol Device:R_Small_US -> LumiCom_TIA:R_Small_US
Changed lines of the file:
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@@
 	)
 	(symbol
-		(lib_id "power:GND")
+		(lib_id "LumiCom_TIA:GND")
 		(at 187.96 121.92 0)
 		(unit 1)
@@
 	)
 	(symbol
-		(lib_id "Connector_Generic:Conn_01x03")
+		(lib_id "LumiCom_TIA:Conn_01x03")
 		(at 208.28 96.52 0)
 		(unit 1)
@@
 			)
 		)
-		(property "Footprint" "Connector_PinHeader_2.54mm:PinHeader_1x03_P2.54mm_Vertical"
+		(property "Footprint" "LumiCom_TIA:PinHeader_1x03_P2.54mm_Vertical"
 			(at 208.28 96.52 0)
 			(effects
@@
 	)
 	(symbol
-		(lib_id "power:VCC")
+		(lib_id "LumiCom_TIA:VCC")
 		(at 144.78 111.76 180)
 		(unit 1)
@@
 	)
 	(symbol
-		(lib_id "Mechanical:MountingHole")
+		(lib_id "LumiCom_TIA:MountingHole")
 		(at 57.15 55.88 0)
 		(unit 1)
@@
 			)
 		)
-		(property "Footprint" "MountingHole:MountingHole_3.2mm_M3_DIN965"
+		(property "Footprint" "LumiCom_TIA:MountingHole_3.2mm_M3_DIN965"
 			(at 57.15 55.88 0)
 			(effects
@@
 	)
 	(symbol
-		(lib_id "power:VCC")
+		(lib_id "LumiCom_TIA:VCC")
 		(at 182.88 43.18 0)
 		(unit 1)
@@
 	)
 	(symbol
-		(lib_id "Device:L_Ferrite_Small")
+		(lib_id "LumiCom_TIA:L_Ferrite_Small")
 		(at 142.24 53.34 90)
 		(unit 1)
@@
 			)
 		)
-		(property "Footprint" "Inductor_SMD:L_0603_1608Metric_Pad1.05x0.95mm_HandSolder"
+		(property "Footprint" "LumiCom_TIA:L_0603_1608Metric_Pad1.05x0.95mm_HandSolder"
 			(at 142.24 53.34 0)
 			(effects
@@
 	)
 	(symbol
-		(lib_id "power:VCC")
+		(lib_id "LumiCom_TIA:VCC")
 		(at 137.16 137.16 0)
 		(unit 1)
@@
 	)
 	(symbol
-		(lib_id "Mechanical:MountingHole")
+		(lib_id "LumiCom_TIA:MountingHole")
 		(at 57.15 62.23 0)
 		(unit 1)
@@
 			)
 		)
-		(property "Footprint" "MountingHole:MountingHole_3.2mm_M3_DIN965"
+		(property "Footprint" "LumiCom_TIA:MountingHole_3.2mm_M3_DIN965"
 			(at 57.15 62.23 0)
 			(effects
@@
 	)
 	(symbol
-		(lib_id "power:GND")
+		(lib_id "LumiCom_TIA:GND")
 		(at 170.18 63.5 0)
 		(unit 1)
@@
 	)
 	(symbol
-		(lib_id "Device:C_Small")
+		(lib_id "LumiCom_TIA:C_Small")
 		(at 170.18 58.42 0)
 		(unit 1)
@@
 			)
 		)
-		(property "Footprint" "Capacitor_SMD:C_0603_1608Metric_Pad1.08x0.95mm_HandSolder"
+		(property "Footprint" "LumiCom_TIA:C_0603_1608Metric_Pad1.08x0.95mm_HandSolder"
 			(at 170.18 58.42 0)
 			(effects
@@
 	)
 	(symbol
-		(lib_id "power:GND")
+		(lib_id "LumiCom_TIA:GND")
 		(at 137.16 149.86 0)
 		(unit 1)
@@
 	)
 	(symbol
-		(lib_id "Device:R_Small_US")
+		(lib_id "LumiCom_TIA:R_Small_US")
 		(at 121.92 116.84 90)
 		(unit 1)
@@
 			)
 		)
-		(property "Footprint" "Resistor_SMD:R_0603_1608Metric_Pad0.98x0.95mm_HandSolder"
+		(property "Footprint" "LumiCom_TIA:R_0603_1608Metric_Pad0.98x0.95mm_HandSolder"
 			(at 121.92 116.84 0)
 			(effects
@@
 	)
 	(symbol
-		(lib_id "Connector:Screw_Terminal_01x02")
+		(lib_id "LumiCom_TIA:Screw_Terminal_01x02")
 		(at 127 55.88 180)
 		(unit 1)
@@
 			)
 		)
-		(property "Footprint" "TerminalBlock_Phoenix:TerminalBlock_Phoenix_MKDS-1,5-2_1x02_P5.00mm_Horizontal"
+		(property "Footprint" "LumiCom_TIA:TerminalBlock_Phoenix_MKDS-1,5-2_1x02_P5.00mm_Horizontal"
 			(at 127 55.88 0)
 			(effects
@@
 	)
 	(symbol
-		(lib_id "Connector:Conn_Coaxial")
+		(lib_id "LumiCom_TIA:Conn_Coaxial")
 		(at 91.44 116.84 0)
 		(mirror y)
@@
 			)
 		)
-		(property "Footprint" "Connector_Coaxial:SMA_Samtec_SMA-J-P-X-ST-EM1_EdgeMount"
+		(property "Footprint" "LumiCom_TIA:SMA_Samtec_SMA-J-P-X-ST-EM1_EdgeMount"
 			(at 91.44 116.84 0)
 			(effects
@@
 	)
 	(symbol
-		(lib_id "Jumper:SolderJumper_2_Open")
+		(lib_id "LumiCom_TIA:SolderJumper_2_Open")
 		(at 132.08 110.49 90)
 		(unit 1)
@@
 		(in_bom yes)
 		(on_board yes)
-		(dnp no)
+		(dnp yes)
 		(fields_autoplaced yes)
 		(property "Reference" "JP1"
@@
 			)
 		)
-		(property "Footprint" "Resistor_SMD:R_0603_1608Metric_Pad0.98x0.95mm_HandSolder"
+		(property "Footprint" "LumiCom_TIA:R_0603_1608Metric_Pad0.98x0.95mm_HandSolder"
 			(at 132.08 110.49 0)
 			(effects
@@
 	)
 	(symbol
-		(lib_id "Device:LED")
+		(lib_id "LumiCom_TIA:LED")
 		(at 195.58 59.69 90)
 		(unit 1)
@@
 			)
 		)
-		(property "Footprint" "LED_SMD:LED_0603_1608Metric"
+		(property "Footprint" "LumiCom_TIA:LED_0603_1608Metric"
 			(at 195.58 59.69 0)
 			(effects
@@
 	)
 	(symbol
-		(lib_id "power:GND")
+		(lib_id "LumiCom_TIA:GND")
 		(at 200.66 104.14 0)
 		(unit 1)
@@
 	)
 	(symbol
-		(lib_id "Device:C_Small")
+		(lib_id "LumiCom_TIA:C_Small")
 		(at 104.14 129.54 0)
 		(mirror y)
@@
 			)
 		)
-		(property "Footprint" "Capacitor_SMD:C_0402_1005Metric_Pad0.74x0.62mm_HandSolder"
+		(property "Footprint" "LumiCom_TIA:C_0402_1005Metric_Pad0.74x0.62mm_HandSolder"
 			(at 104.14 129.54 0)
 			(effects
@@
 	)
 	(symbol
-		(lib_id "Connector:Conn_Coaxial")
+		(lib_id "LumiCom_TIA:Conn_Coaxial")
 		(at 104.14 91.44 0)
 		(mirror y)
@@
 			)
 		)
-		(property "Footprint" "Connector_Coaxial:SMA_Samtec_SMA-J-P-X-ST-EM1_EdgeMount"
+		(property "Footprint" "LumiCom_TIA:SMA_Samtec_SMA-J-P-X-ST-EM1_EdgeMount"
 			(at 104.14 91.44 0)
 			(effects
@@
 	)
 	(symbol
-		(lib_id "power:GND")
+		(lib_id "LumiCom_TIA:GND")
 		(at 157.48 63.5 0)
 		(unit 1)
@@
 	)
 	(symbol
-		(lib_id "power:Earth")
+		(lib_id "LumiCom_TIA:Earth")
 		(at 104.14 101.6 0)
 		(unit 1)
@@
 	)
 	(symbol
-		(lib_id "power:GND")
+		(lib_id "LumiCom_TIA:GND")
 		(at 91.44 121.92 0)
 		(unit 1)
@@
 	)
 	(symbol
-		(lib_id "power:VCC")
+		(lib_id "LumiCom_TIA:VCC")
 		(at 200.66 91.44 0)
 		(mirror y)
@@
 	)
 	(symbol
-		(lib_id "Device:R_Small_US")
+		(lib_id "LumiCom_TIA:R_Small_US")
 		(at 104.14 121.92 0)
 		(unit 1)
@@
 			)
 		)
-		(property "Footprint" "Resistor_SMD:R_0603_1608Metric_Pad0.98x0.95mm_HandSolder"
+		(property "Footprint" "LumiCom_TIA:R_0603_1608Metric_Pad0.98x0.95mm_HandSolder"
 			(at 104.14 121.92 0)
 			(effects
@@
 	)
 	(symbol
-		(lib_id "Device:C_Small")
+		(lib_id "LumiCom_TIA:C_Small")
 		(at 157.48 58.42 0)
 		(unit 1)
@@
 			)
 		)
-		(property "Footprint" "Capacitor_SMD:C_0603_1608Metric_Pad1.08x0.95mm_HandSolder"
+		(property "Footprint" "LumiCom_TIA:C_0603_1608Metric_Pad1.08x0.95mm_HandSolder"
 			(at 157.48 58.42 0)
 			(effects
@@
 	)
 	(symbol
-		(lib_id "Mechanical:MountingHole")
+		(lib_id "LumiCom_TIA:MountingHole")
 		(at 57.15 68.58 0)
 		(unit 1)
@@
 			)
 		)
-		(property "Footprint" "MountingHole:MountingHole_3.2mm_M3_DIN965"
+		(property "Footprint" "LumiCom_TIA:MountingHole_3.2mm_M3_DIN965"
 			(at 57.15 68.58 0)
 			(effects
@@
 	)
 	(symbol
-		(lib_id "Device:C_Small")
+		(lib_id "LumiCom_TIA:C_Small")
 		(at 182.88 58.42 0)
 		(unit 1)
@@
 			)
 		)
-		(property "Footprint" "Capacitor_SMD:C_0603_1608Metric_Pad1.08x0.95mm_HandSolder"
+		(property "Footprint" "LumiCom_TIA:C_0603_1608Metric_Pad1.08x0.95mm_HandSolder"
 			(at 182.88 58.42 0)
 			(effects
@@
 	)
 	(symbol
-		(lib_id "Device:C_Small")
+		(lib_id "LumiCom_TIA:C_Small")
 		(at 226.06 109.22 90)
 		(unit 1)
@@
 			)
 		)
-		(property "Footprint" "Capacitor_SMD:C_0402_1005Metric_Pad0.74x0.62mm_HandSolder"
+		(property "Footprint" "LumiCom_TIA:C_0402_1005Metric_Pad0.74x0.62mm_HandSolder"
 			(at 226.06 109.22 0)
 			(effects
@@
 	)
 	(symbol
-		(lib_id "power:GND")
+		(lib_id "LumiCom_TIA:GND")
 		(at 104.14 134.62 0)
 		(unit 1)
@@
 	)
 	(symbol
-		(lib_id "power:GND")
+		(lib_id "LumiCom_TIA:GND")
 		(at 182.88 63.5 0)
 		(unit 1)
@@
 	)
 	(symbol
-		(lib_id "Device:R_Small_US")
+		(lib_id "LumiCom_TIA:R_Small_US")
 		(at 195.58 68.58 0)
 		(unit 1)
@@
 			)
 		)
-		(property "Footprint" "Resistor_SMD:R_0603_1608Metric_Pad0.98x0.95mm_HandSolder"
+		(property "Footprint" "LumiCom_TIA:R_0603_1608Metric_Pad0.98x0.95mm_HandSolder"
 			(at 195.58 68.58 0)
 			(effects
@@
 	)
 	(symbol
-		(lib_id "Device:C_Small")
+		(lib_id "LumiCom_TIA:C_Small")
 		(at 114.3 116.84 90)
 		(mirror x)
@@
 			)
 		)
-		(property "Footprint" "Capacitor_SMD:C_0402_1005Metric_Pad0.74x0.62mm_HandSolder"
+		(property "Footprint" "LumiCom_TIA:C_0402_1005Metric_Pad0.74x0.62mm_HandSolder"
 			(at 114.3 116.84 0)
 			(effects
@@
 	)
 	(symbol
-		(lib_id "Device:R_Small_US")
+		(lib_id "LumiCom_TIA:R_Small_US")
 		(at 213.36 109.22 90)
 		(unit 1)
@@
 			)
 		)
-		(property "Footprint" "Resistor_SMD:R_0603_1608Metric_Pad0.98x0.95mm_HandSolder"
+		(property "Footprint" "LumiCom_TIA:R_0603_1608Metric_Pad0.98x0.95mm_HandSolder"
 			(at 213.36 109.22 0)
 			(effects
@@
 	)
 	(symbol
-		(lib_id "power:GND")
+		(lib_id "LumiCom_TIA:GND")
 		(at 132.08 58.42 0)
 		(unit 1)
@@
 	)
 	(symbol
-		(lib_id "power:PWR_FLAG")
+		(lib_id "LumiCom_TIA:PWR_FLAG")
 		(at 157.48 53.34 0)
 		(unit 1)
@@
 	)
 	(symbol
-		(lib_id "Connector:Conn_Coaxial")
+		(lib_id "LumiCom_TIA:Conn_Coaxial")
 		(at 246.38 109.22 0)
 		(unit 1)
@@
 			)
 		)
-		(property "Footprint" "Connector_Coaxial:SMA_Samtec_SMA-J-P-X-ST-EM1_EdgeMount"
+		(property "Footprint" "LumiCom_TIA:SMA_Samtec_SMA-J-P-X-ST-EM1_EdgeMount"
 			(at 246.38 109.22 0)
 			(effects
@@
 	)
 	(symbol
-		(lib_id "power:PWR_FLAG")
+		(lib_id "LumiCom_TIA:PWR_FLAG")
 		(at 132.08 58.42 270)
 		(unit 1)
@@
 	)
 	(symbol
-		(lib_id "power:GND")
+		(lib_id "LumiCom_TIA:GND")
 		(at 195.58 71.12 0)
 		(unit 1)
@@
 	)
 	(symbol
-		(lib_id "Device:R_Small_US")
+		(lib_id "LumiCom_TIA:R_Small_US")
 		(at 226.06 116.84 90)
 		(unit 1)
@@
 			)
 		)
-		(property "Footprint" "Resistor_SMD:R_0603_1608Metric_Pad0.98x0.95mm_HandSolder"
+		(property "Footprint" "LumiCom_TIA:R_0603_1608Metric_Pad0.98x0.95mm_HandSolder"
 			(at 226.06 116.84 0)
 			(effects
@@
 	)
 	(symbol
-		(lib_id "Connector_Generic:Conn_01x03")
+		(lib_id "LumiCom_TIA:Conn_01x03")
 		(at 127 142.24 0)
 		(mirror y)
@@
 			)
 		)
-		(property "Footprint" "Connector_PinHeader_2.54mm:PinHeader_1x03_P2.54mm_Vertical"
+		(property "Footprint" "LumiCom_TIA:PinHeader_1x03_P2.54mm_Vertical"
 			(at 127 142.24 0)
 			(effects
@@
 	)
 	(symbol
-		(lib_id "power:GND")
+		(lib_id "LumiCom_TIA:GND")
 		(at 246.38 114.3 0)
 		(unit 1)
