File: Receiver/TIA/LTC6268-10/LTC6268-10.kicad_pcb (KiCad board)
At the start: 4 copper layers, 30 x 40 mm, 29 parts, among them J1 IN, J2 Vout, J3 TEST, J4 OUT, U1 LTC6268-10

Commit message: Vendor project libraries; clean ERC/DRC on all boards
- Copy embedded footprints and symbols into each project's local library
  and repoint FPIDs / lib_ids so every project is self-contained
- Add sym-lib-table for tx_amplifier and preenfasis
- Sync footprint fields with the schematic (parity) and mark LMH34400 JP1 DNP
- Remove dangling copper arc and silkscreen overlap in LTC6268-10
- Fix LED ERC metadata errors
- All 8 boards: ERC and DRC clean (0 errors, 0 warnings)
Parts:
- C1, C3, C7: footprint Capacitor_SMD:C_0402_1005Metric_Pad0.74x0.62mm_HandSolder -> LumiCom_TIA:C_0402_1005Metric_Pad0.74x0.62mm_HandSolder
- C2, C4, C5, C6: footprint Capacitor_SMD:C_0603_1608Metric_Pad1.08x0.95mm_HandSolder -> LumiCom_TIA:C_0603_1608Metric_Pad1.08x0.95mm_HandSolder
- Cf1, Cf2: footprint Capacitor_SMD:C_0402_1005Metric -> LumiCom_TIA:C_0402_1005Metric
- D1: footprint LED_SMD:LED_0603_1608Metric -> LumiCom_TIA:LED_0603_1608Metric
- H1, H2, H3: footprint MountingHole:MountingHole_3.2mm_M3_DIN965 -> LumiCom_TIA:MountingHole_3.2mm_M3_DIN965
- J1, J3, J4: footprint Connector_Coaxial:SMA_Samtec_SMA-J-P-X-ST-EM1_EdgeMount -> LumiCom_TIA:SMA_Samtec_SMA-J-P-X-ST-EM1_EdgeMount
- J2: footprint TerminalBlock_Phoenix:TerminalBlock_Phoenix_MKDS-1,5-2_1x02_P5.00mm_Horizontal -> LumiCom_TIA:TerminalBlock_Phoenix_MKDS-1,5-2_1x02_P5.00mm_Horizontal
- JP1, R1, R2, R3, R4, R5, R6, R7: footprint Resistor_SMD:R_0603_1608Metric_Pad0.98x0.95mm_HandSolder -> LumiCom_TIA:R_0603_1608Metric_Pad0.98x0.95mm_HandSolder
- L1: value Ferrite Beads 220 OHM -> Ferrite Beads 220 OHM; footprint Inductor_SMD:L_0603_1608Metric_Pad1.05x0.95mm_HandSolder -> LumiCom_TIA:L_0603_1608Metric_Pad1.05x0.95mm_HandSolder
- Rf1: footprint Resistor_SMD:R_0402_1005Metric -> LumiCom_TIA:R_0402_1005Metric
- SD_L1: footprint Connector_PinHeader_2.54mm:PinHeader_1x03_P2.54mm_Vertical -> LumiCom_TIA:PinHeader_1x03_P2.54mm_Vertical
