File: Transmitter/AMP/tx_amplifier.kicad_sch (KiCad schematic)
At the start: 20 parts, among them J1 Conn_Coaxial, J2 Conn_Coaxial, J3 Screw_Terminal_01x02, Q1 BFR740L3RH

Commit message: Vendor project libraries; clean ERC/DRC on all boards
- Copy embedded footprints and symbols into each project's local library
  and repoint FPIDs / lib_ids so every project is self-contained
- Add sym-lib-table for tx_amplifier and preenfasis
- Sync footprint fields with the schematic (parity) and mark LMH34400 JP1 DNP
- Remove dangling copper arc and silkscreen overlap in LTC6268-10
- Fix LED ERC metadata errors
- All 8 boards: ERC and DRC clean (0 errors, 0 warnings)
Parts:
- C1, C2, C3, C4, C5, C6: footprint Capacitor_SMD:C_0603_1608Metric_Pad1.08x0.95mm_HandSolder -> vlc:C_0603_1608Metric_Pad1.08x0.95mm_HandSolder; symbol Device:C -> tx_amplifier:C
- H1, H2, H3, H4: footprint MountingHole:MountingHole_3.2mm_M3_ISO7380 -> vlc:MountingHole_3.2mm_M3_ISO7380; symbol Mechanical:MountingHole -> tx_amplifier:MountingHole
- J1, J2: footprint Connector_Coaxial:SMA_Samtec_SMA-J-P-X-ST-EM1_EdgeMount -> vlc:SMA_Samtec_SMA-J-P-X-ST-EM1_EdgeMount; symbol Connector:Conn_Coaxial -> tx_amplifier:Conn_Coaxial
- J3: footprint TerminalBlock:TerminalBlock_bornier-2_P5.08mm -> vlc:TerminalBlock_bornier-2_P5.08mm; symbol Connector:Screw_Terminal_01x02 -> tx_amplifier:Screw_Terminal_01x02
- L1, L2: footprint Inductor_SMD:L_0603_1608Metric_Pad1.05x0.95mm_HandSolder -> vlc:L_0603_1608Metric_Pad1.05x0.95mm_HandSolder; symbol Device:L -> tx_amplifier:L
- Q1: symbol Device:Q_NPN_BCE -> tx_amplifier:Q_NPN_BCE
- R1, R3: footprint Resistor_SMD:R_1206_3216Metric_Pad1.30x1.75mm_HandSolder -> vlc:R_1206_3216Metric_Pad1.30x1.75mm_HandSolder; symbol Device:R_US -> tx_amplifier:R_US
- R2, R4: footprint Resistor_SMD:R_0603_1608Metric_Pad0.98x0.95mm_HandSolder -> vlc:R_0603_1608Metric_Pad0.98x0.95mm_HandSolder; symbol Device:R_US -> tx_amplifier:R_US
Changed lines of the file:
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@@
 	)
 	(symbol
-		(lib_id "Device:C")
+		(lib_id "tx_amplifier:C")
 		(at 66.04 100.33 90)
 		(unit 1)
@@
 			)
 		)
-		(property "Footprint" "Capacitor_SMD:C_0603_1608Metric_Pad1.08x0.95mm_HandSolder"
+		(property "Footprint" "vlc:C_0603_1608Metric_Pad1.08x0.95mm_HandSolder"
 			(at 69.85 99.3648 0)
 			(effects
@@
 	)
 	(symbol
-		(lib_id "Device:C")
+		(lib_id "tx_amplifier:C")
 		(at 135.89 72.39 90)
 		(unit 1)
@@
 			)
 		)
-		(property "Footprint" "Capacitor_SMD:C_0603_1608Metric_Pad1.08x0.95mm_HandSolder"
+		(property "Footprint" "vlc:C_0603_1608Metric_Pad1.08x0.95mm_HandSolder"
 			(at 139.7 71.4248 0)
 			(effects
@@
 	)
 	(symbol
-		(lib_id "Device:C")
+		(lib_id "tx_amplifier:C")
 		(at 93.98 91.44 90)
 		(unit 1)
@@
 			)
 		)
-		(property "Footprint" "Capacitor_SMD:C_0603_1608Metric_Pad1.08x0.95mm_HandSolder"
+		(property "Footprint" "vlc:C_0603_1608Metric_Pad1.08x0.95mm_HandSolder"
 			(at 97.79 90.4748 0)
 			(effects
@@
 	)
 	(symbol
-		(lib_id "Device:C")
+		(lib_id "tx_amplifier:C")
 		(at 153.67 91.44 90)
 		(unit 1)
@@
 			)
 		)
-		(property "Footprint" "Capacitor_SMD:C_0603_1608Metric_Pad1.08x0.95mm_HandSolder"
+		(property "Footprint" "vlc:C_0603_1608Metric_Pad1.08x0.95mm_HandSolder"
 			(at 157.48 90.4748 0)
 			(effects
@@
 	)
 	(symbol
-		(lib_id "Device:R_US")
+		(lib_id "tx_amplifier:R_US")
 		(at 120.65 64.77 180)
 		(unit 1)
@@
 			)
 		)
-		(property "Footprint" "Resistor_SMD:R_1206_3216Metric_Pad1.30x1.75mm_HandSolder"
+		(property "Footprint" "vlc:R_1206_3216Metric_Pad1.30x1.75mm_HandSolder"
 			(at 119.634 64.516 90)
 			(effects
@@
 	)
 	(symbol
-		(lib_id "Device:R_US")
+		(lib_id "tx_amplifier:R_US")
 		(at 81.28 91.44 270)
 		(unit 1)
@@
 			)
 		)
-		(property "Footprint" "Resistor_SMD:R_0603_1608Metric_Pad0.98x0.95mm_HandSolder"
+		(property "Footprint" "vlc:R_0603_1608Metric_Pad0.98x0.95mm_HandSolder"
 			(at 81.026 92.456 90)
 			(effects
@@
 	)
 	(symbol
-		(lib_id "Device:R_US")
+		(lib_id "tx_amplifier:R_US")
 		(at 120.65 82.55 180)
 		(unit 1)
@@
 			)
 		)
-		(property "Footprint" "Resistor_SMD:R_1206_3216Metric_Pad1.30x1.75mm_HandSolder"
+		(property "Footprint" "vlc:R_1206_3216Metric_Pad1.30x1.75mm_HandSolder"
 			(at 119.634 82.296 90)
 			(effects
@@
 	)
 	(symbol
-		(lib_id "Connector:Conn_Coaxial")
+		(lib_id "tx_amplifier:Conn_Coaxial")
 		(at 53.34 100.33 0)
 		(mirror y)
@@
 			)
 		)
-		(property "Footprint" "Connector_Coaxial:SMA_Samtec_SMA-J-P-X-ST-EM1_EdgeMount"
+		(property "Footprint" "vlc:SMA_Samtec_SMA-J-P-X-ST-EM1_EdgeMount"
 			(at 53.34 100.33 0)
 			(effects
@@
 	)
 	(symbol
-		(lib_id "power:GND")
+		(lib_id "tx_amplifier:GND")
 		(at 24.13 29.21 0)
 		(unit 1)
@@
 	)
 	(symbol
-		(lib_id "Mechanical:MountingHole")
+		(lib_id "tx_amplifier:MountingHole")
 		(at 58.42 24.13 0)
 		(unit 1)
@@
 			)
 		)
-		(property "Footprint" "MountingHole:MountingHole_3.2mm_M3_ISO7380"
+		(property "Footprint" "vlc:MountingHole_3.2mm_M3_ISO7380"
 			(at 58.42 24.13 0)
 			(effects
@@
 	)
 	(symbol
-		(lib_id "Connector:Conn_Coaxial")
+		(lib_id "tx_amplifier:Conn_Coaxial")
 		(at 165.1 91.44 0)
 		(unit 1)
@@
 			)
 		)
-		(property "Footprint" "Connector_Coaxial:SMA_Samtec_SMA-J-P-X-ST-EM1_EdgeMount"
+		(property "Footprint" "vlc:SMA_Samtec_SMA-J-P-X-ST-EM1_EdgeMount"
 			(at 165.1 91.44 0)
 			(effects
@@
 	)
 	(symbol
-		(lib_id "power:+3.3V")
+		(lib_id "tx_amplifier:+3.3V")
 		(at 97.79 21.59 0)
 		(unit 1)
@@
 	)
 	(symbol
-		(lib_id "Connector:Screw_Terminal_01x02")
+		(lib_id "tx_amplifier:Screw_Terminal_01x02")
 		(at 80.01 24.13 0)
 		(mirror y)
@@
 			)
 		)
-		(property "Footprint" "TerminalBlock:TerminalBlock_bornier-2_P5.08mm"
+		(property "Footprint" "vlc:TerminalBlock_bornier-2_P5.08mm"
 			(at 80.01 24.13 0)
 			(effects
@@
 	)
 	(symbol
-		(lib_id "Mechanical:MountingHole")
+		(lib_id "tx_amplifier:MountingHole")
 		(at 48.26 24.13 0)
 		(unit 1)
@@
 			)
 		)
-		(property "Footprint" "MountingHole:MountingHole_3.2mm_M3_ISO7380"
+		(property "Footprint" "vlc:MountingHole_3.2mm_M3_ISO7380"
 			(at 48.26 24.13 0)
 			(effects
@@
 	)
 	(symbol
-		(lib_id "power:GND")
+		(lib_id "tx_amplifier:GND")
 		(at 53.34 121.92 0)
 		(unit 1)
@@
 	)
 	(symbol
-		(lib_id "Device:R_US")
+		(lib_id "tx_amplifier:R_US")
 		(at 73.66 80.01 180)
 		(unit 1)
@@
 			)
 		)
-		(property "Footprint" "Resistor_SMD:R_0603_1608Metric_Pad0.98x0.95mm_HandSolder"
+		(property "Footprint" "vlc:R_0603_1608Metric_Pad0.98x0.95mm_HandSolder"
 			(at 72.644 79.756 90)
 			(effects
@@
 	)
 	(symbol
-		(lib_id "Device:C")
+		(lib_id "tx_amplifier:C")
 		(at 139.7 111.76 180)
 		(unit 1)
@@
 			)
 		)
-		(property "Footprint" "Capacitor_SMD:C_0603_1608Metric_Pad1.08x0.95mm_HandSolder"
+		(property "Footprint" "vlc:C_0603_1608Metric_Pad1.08x0.95mm_HandSolder"
 			(at 138.7348 107.95 0)
 			(effects
@@
 	)
 	(symbol
-		(lib_id "Device:C")
+		(lib_id "tx_amplifier:C")
 		(at 120.65 105.41 180)
 		(unit 1)
@@
 			)
 		)
-		(property "Footprint" "Capacitor_SMD:C_0603_1608Metric_Pad1.08x0.95mm_HandSolder"
+		(property "Footprint" "vlc:C_0603_1608Metric_Pad1.08x0.95mm_HandSolder"
 			(at 119.6848 101.6 0)
 			(effects
@@
 	)
 	(symbol
-		(lib_id "power:+3.3V")
+		(lib_id "tx_amplifier:+3.3V")
 		(at 34.29 24.13 0)
 		(unit 1)
@@
 	)
 	(symbol
-		(lib_id "power:GND")
+		(lib_id "tx_amplifier:GND")
 		(at 97.79 26.67 0)
 		(unit 1)
@@
 	)
 	(symbol
-		(lib_id "Device:L")
+		(lib_id "tx_amplifier:L")
 		(at 130.81 91.44 90)
 		(unit 1)
@@
 			)
 		)
-		(property "Footprint" "Inductor_SMD:L_0603_1608Metric_Pad1.05x0.95mm_HandSolder"
+		(property "Footprint" "vlc:L_0603_1608Metric_Pad1.05x0.95mm_HandSolder"
 			(at 130.81 91.44 0)
 			(effects
@@
 	)
 	(symbol
-		(lib_id "Device:L")
+		(lib_id "tx_amplifier:L")
 		(at 139.7 100.33 0)
 		(unit 1)
@@
 			)
 		)
-		(property "Footprint" "Inductor_SMD:L_0603_1608Metric_Pad1.05x0.95mm_HandSolder"
+		(property "Footprint" "vlc:L_0603_1608Metric_Pad1.05x0.95mm_HandSolder"
 			(at 139.7 100.33 0)
 			(effects
@@
 	)
 	(symbol
-		(lib_id "power:+3.3V")
+		(lib_id "tx_amplifier:+3.3V")
 		(at 120.65 57.15 0)
 		(unit 1)
@@
 	)
 	(symbol
-		(lib_id "power:GND")
+		(lib_id "tx_amplifier:GND")
 		(at 144.78 72.39 0)
 		(unit 1)
@@
 	)
 	(symbol
-		(lib_id "Mechanical:MountingHole")
+		(lib_id "tx_amplifier:MountingHole")
 		(at 58.42 17.78 0)
 		(unit 1)
@@
 			)
 		)
-		(property "Footprint" "MountingHole:MountingHole_3.2mm_M3_ISO7380"
+		(property "Footprint" "vlc:MountingHole_3.2mm_M3_ISO7380"
 			(at 58.42 17.78 0)
 			(effects
@@
 	)
 	(symbol
-		(lib_id "power:PWR_FLAG")
+		(lib_id "tx_amplifier:PWR_FLAG")
 		(at 34.29 29.21 180)
 		(unit 1)
@@
 	)
 	(symbol
-		(lib_id "power:PWR_FLAG")
+		(lib_id "tx_amplifier:PWR_FLAG")
 		(at 24.13 24.13 0)
 		(unit 1)
@@
 	)
 	(symbol
-		(lib_id "Device:Q_NPN_BCE")
+		(lib_id "tx_amplifier:Q_NPN_BCE")
 		(at 99.06 100.33 0)
 		(unit 1)
@@
 	)
 	(symbol
-		(lib_id "Mechanical:MountingHole")
+		(lib_id "tx_amplifier:MountingHole")
 		(at 48.26 17.78 0)
 		(unit 1)
@@
 			)
 		)
-		(property "Footprint" "MountingHole:MountingHole_3.2mm_M3_ISO7380"
+		(property "Footprint" "vlc:MountingHole_3.2mm_M3_ISO7380"
 			(at 48.26 17.78 0)
 			(effects
