File: Transmitter/FCA/Amplifier.kicad_sch (KiCad schematic)
At the start: 29 parts, among them J2 IN_B, J3 IN_A, J4 OUT_B, J5 OUT_A, U1 OPA2675

Commit message: Vendor project libraries; clean ERC/DRC on all boards
- Copy embedded footprints and symbols into each project's local library
  and repoint FPIDs / lib_ids so every project is self-contained
- Add sym-lib-table for tx_amplifier and preenfasis
- Sync footprint fields with the schematic (parity) and mark LMH34400 JP1 DNP
- Remove dangling copper arc and silkscreen overlap in LTC6268-10
- Fix LED ERC metadata errors
- All 8 boards: ERC and DRC clean (0 errors, 0 warnings)
Parts:
- C10, C3, C4, C5, C6, C7, C8, C9: symbol Device:C_Small -> Lumicom_Transmitter:C_Small
- J2, J3, J4, J5: symbol Connector:Conn_Coaxial -> Lumicom_Transmitter:Conn_Coaxial
- JP_A1, JP_A2: footprint Connector_PinHeader_2.54mm:PinHeader_1x03_P2.54mm_Vertical -> LumiCom_Transmitter:PinHeader_1x03_P2.54mm_Vertical; symbol Jumper:Jumper_3_Bridged12 -> Lumicom_Transmitter:Jumper_3_Bridged12
- R1, R10, R11, R12, R2, R3, R4, R5, R6, R7, R8, R9: footprint Resistor_SMD:R_0603_1608Metric -> LumiCom_Transmitter:R_0603_1608Metric; symbol Device:R_Small_US -> Lumicom_Transmitter:R_Small_US
- R13, R14: symbol Device:R_Small_US -> Lumicom_Transmitter:R_Small_US
Changed lines of the file:
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@@
 	)
 	(symbol
-		(lib_id "Device:R_Small_US")
+		(lib_id "Lumicom_Transmitter:R_Small_US")
 		(at 228.6 104.14 90)
 		(unit 1)
@@
 	)
 	(symbol
-		(lib_id "power:GND")
+		(lib_id "Lumicom_Transmitter:GND")
 		(at 176.53 143.51 0)
 		(unit 1)
@@
 	)
 	(symbol
-		(lib_id "power:GND")
+		(lib_id "Lumicom_Transmitter:GND")
 		(at 163.83 143.51 0)
 		(unit 1)
@@
 	)
 	(symbol
-		(lib_id "Device:C_Small")
+		(lib_id "Lumicom_Transmitter:C_Small")
 		(at 214.63 81.28 90)
 		(unit 1)
@@
 	)
 	(symbol
-		(lib_id "power:GND")
+		(lib_id "Lumicom_Transmitter:GND")
 		(at 138.43 143.51 0)
 		(unit 1)
@@
 	)
 	(symbol
-		(lib_id "Device:R_Small_US")
+		(lib_id "Lumicom_Transmitter:R_Small_US")
 		(at 101.6 69.85 0)
 		(unit 1)
@@
 			)
 		)
-		(property "Footprint" "Resistor_SMD:R_0603_1608Metric"
+		(property "Footprint" "LumiCom_Transmitter:R_0603_1608Metric"
 			(at 101.6 69.85 0)
 			(effects
@@
 	)
 	(symbol
-		(lib_id "Device:C_Small")
+		(lib_id "Lumicom_Transmitter:C_Small")
 		(at 95.25 133.35 180)
 		(unit 1)
@@
 	)
 	(symbol
-		(lib_id "Device:R_Small_US")
+		(lib_id "Lumicom_Transmitter:R_Small_US")
 		(at 180.34 119.38 90)
 		(unit 1)
@@
 			)
 		)
-		(property "Footprint" "Resistor_SMD:R_0603_1608Metric"
+		(property "Footprint" "LumiCom_Transmitter:R_0603_1608Metric"
 			(at 180.34 119.38 0)
 			(effects
@@
 	)
 	(symbol
-		(lib_id "Connector:Conn_Coaxial")
+		(lib_id "Lumicom_Transmitter:Conn_Coaxial")
 		(at 254 81.28 0)
 		(unit 1)
@@
 	)
 	(symbol
-		(lib_id "Device:R_Small_US")
+		(lib_id "Lumicom_Transmitter:R_Small_US")
 		(at 101.6 57.15 0)
 		(unit 1)
@@
 			)
 		)
-		(property "Footprint" "Resistor_SMD:R_0603_1608Metric"
+		(property "Footprint" "LumiCom_Transmitter:R_0603_1608Metric"
 			(at 101.6 57.15 0)
 			(effects
@@
 	)
 	(symbol
-		(lib_id "Jumper:Jumper_3_Bridged12")
+		(lib_id "Lumicom_Transmitter:Jumper_3_Bridged12")
 		(at 149.86 45.72 0)
 		(unit 1)
@@
 			)
 		)
-		(property "Footprint" "Connector_PinHeader_2.54mm:PinHeader_1x03_P2.54mm_Vertical"
+		(property "Footprint" "LumiCom_Transmitter:PinHeader_1x03_P2.54mm_Vertical"
 			(at 149.86 45.72 0)
 			(effects
@@
 	)
 	(symbol
-		(lib_id "power:VCC")
+		(lib_id "Lumicom_Transmitter:VCC")
 		(at 101.6 50.8 0)
 		(unit 1)
@@
 	)
 	(symbol
-		(lib_id "Connector:Conn_Coaxial")
+		(lib_id "Lumicom_Transmitter:Conn_Coaxial")
 		(at 82.55 63.5 0)
 		(mirror y)
@@
 	)
 	(symbol
-		(lib_id "power:GND")
+		(lib_id "Lumicom_Transmitter:GND")
 		(at 165.1 114.3 0)
 		(unit 1)
@@
 	)
 	(symbol
-		(lib_id "power:GND")
+		(lib_id "Lumicom_Transmitter:GND")
 		(at 138.43 45.72 0)
 		(mirror y)
@@
 	)
 	(symbol
-		(lib_id "Device:R_Small_US")
+		(lib_id "Lumicom_Transmitter:R_Small_US")
 		(at 76.2 120.65 0)
 		(unit 1)
@@
 			)
 		)
-		(property "Footprint" "Resistor_SMD:R_0603_1608Metric"
+		(property "Footprint" "LumiCom_Transmitter:R_0603_1608Metric"
 			(at 76.2 120.65 0)
 			(effects
@@
 	)
 	(symbol
-		(lib_id "Device:R_Small_US")
+		(lib_id "Lumicom_Transmitter:R_Small_US")
 		(at 114.3 69.85 0)
 		(unit 1)
@@
 			)
 		)
-		(property "Footprint" "Resistor_SMD:R_0603_1608Metric"
+		(property "Footprint" "LumiCom_Transmitter:R_0603_1608Metric"
 			(at 114.3 69.85 0)
 			(effects
@@
 	)
 	(symbol
-		(lib_id "Device:R_Small_US")
+		(lib_id "Lumicom_Transmitter:R_Small_US")
 		(at 151.13 135.89 180)
 		(unit 1)
@@
 			)
 		)
-		(property "Footprint" "Resistor_SMD:R_0603_1608Metric"
+		(property "Footprint" "LumiCom_Transmitter:R_0603_1608Metric"
 			(at 151.13 135.89 0)
 			(effects
@@
 	)
 	(symbol
-		(lib_id "Device:R_Small_US")
+		(lib_id "Lumicom_Transmitter:R_Small_US")
 		(at 113.03 106.68 180)
 		(unit 1)
@@
 			)
 		)
-		(property "Footprint" "Resistor_SMD:R_0603_1608Metric"
+		(property "Footprint" "LumiCom_Transmitter:R_0603_1608Metric"
 			(at 113.03 106.68 0)
 			(effects
@@
 	)
 	(symbol
-		(lib_id "Jumper:Jumper_3_Bridged12")
+		(lib_id "Lumicom_Transmitter:Jumper_3_Bridged12")
 		(at 176.53 45.72 0)
 		(unit 1)
@@
 			)
 		)
-		(property "Footprint" "Connector_PinHeader_2.54mm:PinHeader_1x03_P2.54mm_Vertical"
+		(property "Footprint" "LumiCom_Transmitter:PinHeader_1x03_P2.54mm_Vertical"
 			(at 176.53 45.72 0)
 			(effects
@@
 	)
 	(symbol
-		(lib_id "Device:R_Small_US")
+		(lib_id "Lumicom_Transmitter:R_Small_US")
 		(at 125.73 106.68 180)
 		(unit 1)
@@
 			)
 		)
-		(property "Footprint" "Resistor_SMD:R_0603_1608Metric"
+		(property "Footprint" "LumiCom_Transmitter:R_0603_1608Metric"
 			(at 125.73 106.68 0)
 			(effects
@@
 	)
 	(symbol
-		(lib_id "Device:R_Small_US")
+		(lib_id "Lumicom_Transmitter:R_Small_US")
 		(at 191.77 128.27 90)
 		(unit 1)
@@
 			)
 		)
-		(property "Footprint" "Resistor_SMD:R_0603_1608Metric"
+		(property "Footprint" "LumiCom_Transmitter:R_0603_1608Metric"
 			(at 191.77 128.27 0)
 			(effects
@@
 	)
 	(symbol
-		(lib_id "power:GND")
+		(lib_id "Lumicom_Transmitter:GND")
 		(at 114.3 82.55 0)
 		(unit 1)
@@
 	)
 	(symbol
-		(lib_id "power:GND")
+		(lib_id "Lumicom_Transmitter:GND")
 		(at 76.2 127 0)
 		(unit 1)
@@
 	)
 	(symbol
-		(lib_id "power:GND")
+		(lib_id "Lumicom_Transmitter:GND")
 		(at 151.13 143.51 0)
 		(unit 1)
@@
 	)
 	(symbol
-		(lib_id "power:GND")
+		(lib_id "Lumicom_Transmitter:GND")
 		(at 190.5 45.72 0)
 		(unit 1)
@@
 	)
 	(symbol
-		(lib_id "Device:R_Small_US")
+		(lib_id "Lumicom_Transmitter:R_Small_US")
 		(at 176.53 135.89 180)
 		(unit 1)
@@
 			)
 		)
-		(property "Footprint" "Resistor_SMD:R_0603_1608Metric"
+		(property "Footprint" "LumiCom_Transmitter:R_0603_1608Metric"
 			(at 176.53 135.89 0)
 			(effects
@@
 	)
 	(symbol
-		(lib_id "Device:C_Small")
+		(lib_id "Lumicom_Transmitter:C_Small")
 		(at 69.85 114.3 90)
 		(unit 1)
@@
 	)
 	(symbol
-		(lib_id "power:GND")
+		(lib_id "Lumicom_Transmitter:GND")
 		(at 82.55 69.85 0)
 		(unit 1)
@@
 	)
 	(symbol
-		(lib_id "power:GND")
+		(lib_id "Lumicom_Transmitter:GND")
 		(at 101.6 76.2 0)
 		(unit 1)
@@
 	)
 	(symbol
-		(lib_id "Connector:Conn_Coaxial")
+		(lib_id "Lumicom_Transmitter:Conn_Coaxial")
 		(at 57.15 114.3 0)
 		(mirror y)
@@
 	)
 	(symbol
-		(lib_id "power:GND")
+		(lib_id "Lumicom_Transmitter:GND")
 		(at 95.25 139.7 0)
 		(unit 1)
@@
 	)
 	(symbol
-		(lib_id "Device:R_Small_US")
+		(lib_id "Lumicom_Transmitter:R_Small_US")
 		(at 76.2 107.95 0)
 		(unit 1)
@@
 			)
 		)
-		(property "Footprint" "Resistor_SMD:R_0603_1608Metric"
+		(property "Footprint" "LumiCom_Transmitter:R_0603_1608Metric"
 			(at 76.2 107.95 0)
 			(effects
@@
 	)
 	(symbol
-		(lib_id "power:VCC")
+		(lib_id "Lumicom_Transmitter:VCC")
 		(at 163.83 34.29 0)
 		(unit 1)
@@
 	)
 	(symbol
-		(lib_id "Device:R_Small_US")
+		(lib_id "Lumicom_Transmitter:R_Small_US")
 		(at 227.33 81.28 90)
 		(unit 1)
@@
 	)
 	(symbol
-		(lib_id "power:VCC")
+		(lib_id "Lumicom_Transmitter:VCC")
 		(at 76.2 101.6 0)
 		(unit 1)
@@
 	)
 	(symbol
-		(lib_id "power:GND")
+		(lib_id "Lumicom_Transmitter:GND")
 		(at 57.15 120.65 0)
 		(unit 1)
@@
 	)
 	(symbol
-		(lib_id "Device:C_Small")
+		(lib_id "Lumicom_Transmitter:C_Small")
 		(at 215.9 104.14 90)
 		(unit 1)
@@
 	)
 	(symbol
-		(lib_id "power:GND")
+		(lib_id "Lumicom_Transmitter:GND")
 		(at 171.45 114.3 0)
 		(unit 1)
@@
 	)
 	(symbol
-		(lib_id "power:GND")
+		(lib_id "Lumicom_Transmitter:GND")
 		(at 187.325 104.775 0)
 		(unit 1)
@@
 	)
 	(symbol
-		(lib_id "Connector:Conn_Coaxial")
+		(lib_id "Lumicom_Transmitter:Conn_Coaxial")
 		(at 252.73 104.14 0)
 		(unit 1)
@@
 	)
 	(symbol
-		(lib_id "power:GND")
+		(lib_id "Lumicom_Transmitter:GND")
 		(at 142.24 106.68 0)
 		(unit 1)
@@
 	)
 	(symbol
-		(lib_id "Device:C_Small")
+		(lib_id "Lumicom_Transmitter:C_Small")
 		(at 138.43 135.89 0)
 		(unit 1)
@@
 	)
 	(symbol
-		(lib_id "Device:R_Small_US")
+		(lib_id "Lumicom_Transmitter:R_Small_US")
 		(at 95.25 123.825 0)
 		(unit 1)
@@
 			)
 		)
-		(property "Footprint" "Resistor_SMD:R_0603_1608Metric"
+		(property "Footprint" "LumiCom_Transmitter:R_0603_1608Metric"
 			(at 95.25 123.825 0)
 			(effects
@@
 	)
 	(symbol
-		(lib_id "Device:C_Small")
+		(lib_id "Lumicom_Transmitter:C_Small")
 		(at 163.83 135.89 0)
 		(unit 1)
@@
 	)
 	(symbol
-		(lib_id "power:GND")
+		(lib_id "Lumicom_Transmitter:GND")
 		(at 254 87.63 0)
 		(unit 1)
@@
 	)
 	(symbol
-		(lib_id "Device:C_Small")
+		(lib_id "Lumicom_Transmitter:C_Small")
 		(at 95.25 63.5 90)
 		(unit 1)
@@
 	)
 	(symbol
-		(lib_id "Device:C_Small")
+		(lib_id "Lumicom_Transmitter:C_Small")
 		(at 114.3 76.2 180)
 		(unit 1)
@@
 	)
 	(symbol
-		(lib_id "power:GND")
+		(lib_id "Lumicom_Transmitter:GND")
 		(at 252.73 111.76 0)
 		(unit 1)
@@
 	)
 	(symbol
-		(lib_id "power:GND")
+		(lib_id "Lumicom_Transmitter:GND")
 		(at 158.75 114.3 0)
 		(unit 1)
