File: Transmitter/FCA/Filter.kicad_sch (KiCad schematic)
At the start: 28 parts, among them J6 Conn_Coaxial, J7 Conn_Coaxial, J8 Screw_Terminal_01x02, Q1 NPN

Commit message: Vendor project libraries; clean ERC/DRC on all boards
- Copy embedded footprints and symbols into each project's local library
  and repoint FPIDs / lib_ids so every project is self-contained
- Add sym-lib-table for tx_amplifier and preenfasis
- Sync footprint fields with the schematic (parity) and mark LMH34400 JP1 DNP
- Remove dangling copper arc and silkscreen overlap in LTC6268-10
- Fix LED ERC metadata errors
- All 8 boards: ERC and DRC clean (0 errors, 0 warnings)
Parts:
- C11, C12, C13, C14, C15, C16, C17: symbol Device:C_Small -> Lumicom_Transmitter:C_Small
- J6, J7: symbol Connector:Conn_Coaxial -> Lumicom_Transmitter:Conn_Coaxial
- J8: symbol Connector:Screw_Terminal_01x02 -> Lumicom_Transmitter:Screw_Terminal_01x02
- L1, L2, L3: symbol Device:L_Small -> Lumicom_Transmitter:L_Small
- Q1: symbol Simulation_SPICE:NPN -> Lumicom_Transmitter:NPN
- R15, R16, R17, R18, R19, R20, R21, R22, R23, R24, R25, R26, R27, R28: footprint Resistor_SMD:R_0603_1608Metric -> LumiCom_Transmitter:R_0603_1608Metric; symbol Device:R_Small_US -> Lumicom_Transmitter:R_Small_US
Changed lines of the file:
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@@
 	)
 	(symbol
-		(lib_id "Device:R_Small_US")
+		(lib_id "Lumicom_Transmitter:R_Small_US")
 		(at 127 58.42 0)
 		(mirror x)
@@
 			)
 		)
-		(property "Footprint" "Resistor_SMD:R_0603_1608Metric"
+		(property "Footprint" "LumiCom_Transmitter:R_0603_1608Metric"
 			(at 127 58.42 0)
 			(effects
@@
 	)
 	(symbol
-		(lib_id "Device:R_Small_US")
+		(lib_id "Lumicom_Transmitter:R_Small_US")
 		(at 88.9 76.2 90)
 		(unit 1)
@@
 			)
 		)
-		(property "Footprint" "Resistor_SMD:R_0603_1608Metric"
+		(property "Footprint" "LumiCom_Transmitter:R_0603_1608Metric"
 			(at 88.9 76.2 0)
 			(effects
@@
 	)
 	(symbol
-		(lib_id "Device:R_Small_US")
+		(lib_id "Lumicom_Transmitter:R_Small_US")
 		(at 76.2 76.2 90)
 		(unit 1)
@@
 			)
 		)
-		(property "Footprint" "Resistor_SMD:R_0603_1608Metric"
+		(property "Footprint" "LumiCom_Transmitter:R_0603_1608Metric"
 			(at 76.2 76.2 0)
 			(effects
@@
 	)
 	(symbol
-		(lib_id "Simulation_SPICE:NPN")
+		(lib_id "Lumicom_Transmitter:NPN")
 		(at 137.16 76.2 0)
 		(unit 1)
@@
 	)
 	(symbol
-		(lib_id "Device:R_Small_US")
+		(lib_id "Lumicom_Transmitter:R_Small_US")
 		(at 82.55 96.52 0)
 		(unit 1)
@@
 			)
 		)
-		(property "Footprint" "Resistor_SMD:R_0603_1608Metric"
+		(property "Footprint" "LumiCom_Transmitter:R_0603_1608Metric"
 			(at 82.55 96.52 0)
 			(effects
@@
 	)
 	(symbol
-		(lib_id "Device:R_Small_US")
+		(lib_id "Lumicom_Transmitter:R_Small_US")
 		(at 127 91.44 180)
 		(unit 1)
@@
 			)
 		)
-		(property "Footprint" "Resistor_SMD:R_0603_1608Metric"
+		(property "Footprint" "LumiCom_Transmitter:R_0603_1608Metric"
 			(at 127 91.44 0)
 			(effects
@@
 	)
 	(symbol
-		(lib_id "Device:C_Small")
+		(lib_id "Lumicom_Transmitter:C_Small")
 		(at 76.2 109.22 180)
 		(unit 1)
@@
 	)
 	(symbol
-		(lib_id "power:GND")
+		(lib_id "Lumicom_Transmitter:GND")
 		(at 82.55 119.38 0)
 		(unit 1)
@@
 	)
 	(symbol
-		(lib_id "power:GND")
+		(lib_id "Lumicom_Transmitter:GND")
 		(at 139.7 107.95 0)
 		(unit 1)
@@
 	)
 	(symbol
-		(lib_id "Device:R_Small_US")
+		(lib_id "Lumicom_Transmitter:R_Small_US")
 		(at 107.95 93.98 180)
 		(unit 1)
@@
 			)
 		)
-		(property "Footprint" "Resistor_SMD:R_0603_1608Metric"
+		(property "Footprint" "LumiCom_Transmitter:R_0603_1608Metric"
 			(at 107.95 93.98 0)
 			(effects
@@
 	)
 	(symbol
-		(lib_id "Device:C_Small")
+		(lib_id "Lumicom_Transmitter:C_Small")
 		(at 152.4 48.26 180)
 		(unit 1)
@@
 	)
 	(symbol
-		(lib_id "Device:C_Small")
+		(lib_id "Lumicom_Transmitter:C_Small")
 		(at 107.95 85.09 180)
 		(unit 1)
@@
 	)
 	(symbol
-		(lib_id "Device:R_Small_US")
+		(lib_id "Lumicom_Transmitter:R_Small_US")
 		(at 171.45 69.85 270)
 		(unit 1)
@@
 			)
 		)
-		(property "Footprint" "Resistor_SMD:R_0603_1608Metric"
+		(property "Footprint" "LumiCom_Transmitter:R_0603_1608Metric"
 			(at 171.45 69.85 0)
 			(effects
@@
 	)
 	(symbol
-		(lib_id "Device:R_Small_US")
+		(lib_id "Lumicom_Transmitter:R_Small_US")
 		(at 87.63 41.91 270)
 		(unit 1)
@@
 			)
 		)
-		(property "Footprint" "Resistor_SMD:R_0603_1608Metric"
+		(property "Footprint" "LumiCom_Transmitter:R_0603_1608Metric"
 			(at 87.63 41.91 0)
 			(effects
@@
 	)
 	(symbol
-		(lib_id "power:GND")
+		(lib_id "Lumicom_Transmitter:GND")
 		(at 203.2 74.93 0)
 		(unit 1)
@@
 	)
 	(symbol
-		(lib_id "Connector:Conn_Coaxial")
+		(lib_id "Lumicom_Transmitter:Conn_Coaxial")
 		(at 44.45 76.2 0)
 		(mirror y)
@@
 	)
 	(symbol
-		(lib_id "Connector:Conn_Coaxial")
+		(lib_id "Lumicom_Transmitter:Conn_Coaxial")
 		(at 203.2 69.85 0)
 		(unit 1)
@@
 	)
 	(symbol
-		(lib_id "Device:L_Small")
+		(lib_id "Lumicom_Transmitter:L_Small")
 		(at 78.74 41.91 90)
 		(unit 1)
@@
 	)
 	(symbol
-		(lib_id "Device:R_Small_US")
+		(lib_id "Lumicom_Transmitter:R_Small_US")
 		(at 88.9 109.22 0)
 		(unit 1)
@@
 			)
 		)
-		(property "Footprint" "Resistor_SMD:R_0603_1608Metric"
+		(property "Footprint" "LumiCom_Transmitter:R_0603_1608Metric"
 			(at 88.9 109.22 0)
 			(effects
@@
 	)
 	(symbol
-		(lib_id "Device:C_Small")
+		(lib_id "Lumicom_Transmitter:C_Small")
 		(at 82.55 63.5 90)
 		(unit 1)
@@
 	)
 	(symbol
-		(lib_id "Device:R_Small_US")
+		(lib_id "Lumicom_Transmitter:R_Small_US")
 		(at 82.55 50.8 270)
 		(unit 1)
@@
 			)
 		)
-		(property "Footprint" "Resistor_SMD:R_0603_1608Metric"
+		(property "Footprint" "LumiCom_Transmitter:R_0603_1608Metric"
 			(at 82.55 50.8 0)
 			(effects
@@
 	)
 	(symbol
-		(lib_id "Device:R_Small_US")
+		(lib_id "Lumicom_Transmitter:R_Small_US")
 		(at 139.7 58.42 180)
 		(unit 1)
@@
 			)
 		)
-		(property "Footprint" "Resistor_SMD:R_0603_1608Metric"
+		(property "Footprint" "LumiCom_Transmitter:R_0603_1608Metric"
 			(at 139.7 58.42 0)
 			(effects
@@
 	)
 	(symbol
-		(lib_id "Device:R_Small_US")
+		(lib_id "Lumicom_Transmitter:R_Small_US")
 		(at 139.7 92.71 180)
 		(unit 1)
@@
 			)
 		)
-		(property "Footprint" "Resistor_SMD:R_0603_1608Metric"
+		(property "Footprint" "LumiCom_Transmitter:R_0603_1608Metric"
 			(at 139.7 92.71 0)
 			(effects
@@
 	)
 	(symbol
-		(lib_id "Device:L_Small")
+		(lib_id "Lumicom_Transmitter:L_Small")
 		(at 82.55 88.9 0)
 		(unit 1)
@@
 	)
 	(symbol
-		(lib_id "Device:L_Small")
+		(lib_id "Lumicom_Transmitter:L_Small")
 		(at 152.4 57.15 0)
 		(unit 1)
@@
 	)
 	(symbol
-		(lib_id "Device:C_Small")
+		(lib_id "Lumicom_Transmitter:C_Small")
 		(at 101.6 76.2 90)
 		(unit 1)
@@
 	)
 	(symbol
-		(lib_id "Device:C_Small")
+		(lib_id "Lumicom_Transmitter:C_Small")
 		(at 181.61 69.85 90)
 		(unit 1)
@@
 	)
 	(symbol
-		(lib_id "power:GND")
+		(lib_id "Lumicom_Transmitter:GND")
 		(at 44.45 81.28 0)
 		(unit 1)
@@
 	)
 	(symbol
-		(lib_id "power:GND")
+		(lib_id "Lumicom_Transmitter:GND")
 		(at 190.5 38.1 0)
 		(unit 1)
@@
 	)
 	(symbol
-		(lib_id "Device:R_Small_US")
+		(lib_id "Lumicom_Transmitter:R_Small_US")
 		(at 152.4 64.77 180)
 		(unit 1)
@@
 			)
 		)
-		(property "Footprint" "Resistor_SMD:R_0603_1608Metric"
+		(property "Footprint" "LumiCom_Transmitter:R_0603_1608Metric"
 			(at 152.4 64.77 0)
 			(effects
@@
 	)
 	(symbol
-		(lib_id "Connector:Screw_Terminal_01x02")
+		(lib_id "Lumicom_Transmitter:Screw_Terminal_01x02")
 		(at 207.01 35.56 0)
 		(unit 1)
@@
 	)
 	(symbol
-		(lib_id "Device:C_Small")
+		(lib_id "Lumicom_Transmitter:C_Small")
 		(at 152.4 88.9 180)
 		(unit 1)
@@
 	)
 	(symbol
-		(lib_id "Device:R_Small_US")
+		(lib_id "Lumicom_Transmitter:R_Small_US")
 		(at 152.4 97.79 180)
 		(unit 1)
@@
 			)
 		)
-		(property "Footprint" "Resistor_SMD:R_0603_1608Metric"
+		(property "Footprint" "LumiCom_Transmitter:R_0603_1608Metric"
 			(at 152.4 97.79 0)
 			(effects
