File: Transmitter/FCA/LumiCom_Transmitter.kicad_pcb (KiCad board)
At the start: 4 copper layers, 50 x 42 mm, 38 parts, among them J1 V, J2 IN_B, J3 IN_A, J4 OUT_B, J5 OUT_A, U1 OPA2675

Commit message: Vendor project libraries; clean ERC/DRC on all boards
- Copy embedded footprints and symbols into each project's local library
  and repoint FPIDs / lib_ids so every project is self-contained
- Add sym-lib-table for tx_amplifier and preenfasis
- Sync footprint fields with the schematic (parity) and mark LMH34400 JP1 DNP
- Remove dangling copper arc and silkscreen overlap in LTC6268-10
- Fix LED ERC metadata errors
- All 8 boards: ERC and DRC clean (0 errors, 0 warnings)
Parts:
- C1, C2, C7: footprint Capacitor_SMD:C_0603_1608Metric_Pad1.08x0.95mm_HandSolder -> LumiCom_Transmitter:C_0603_1608Metric_Pad1.08x0.95mm_HandSolder
- C10, C11, C3, C4, C5, C6, C8, C9: footprint Capacitor_SMD:C_0402_1005Metric_Pad0.74x0.62mm_HandSolder -> LumiCom_Transmitter:C_0402_1005Metric_Pad0.74x0.62mm_HandSolder
- D1: value 150060VS75000 -> 150060VS75000
- H1, H2, H3, H4: footprint MountingHole:MountingHole_3.2mm_M3_ISO7380 -> LumiCom_Transmitter:MountingHole_3.2mm_M3_ISO7380
- J1: footprint TerminalBlock_Phoenix:TerminalBlock_Phoenix_MKDS-1,5-2_1x02_P5.00mm_Horizontal -> LumiCom_Transmitter:TerminalBlock_Phoenix_MKDS-1,5-2_1x02_P5.00mm_Horizontal
- J2, J3, J4, J5: footprint Connector_Coaxial:SMA_Samtec_SMA-J-P-X-ST-EM1_EdgeMount -> LumiCom_Transmitter:SMA_Samtec_SMA-J-P-X-ST-EM1_EdgeMount
- JP_A0, JP_A1: footprint Connector_PinHeader_2.54mm:PinHeader_1x03_P2.54mm_Vertical -> LumiCom_Transmitter:PinHeader_1x03_P2.54mm_Vertical
- L1: value Ferrite Beads 220 OHM -> Ferrite Beads 220 OHM; footprint Inductor_SMD:L_0603_1608Metric_Pad1.05x0.95mm_HandSolder -> LumiCom_Transmitter:L_0603_1608Metric_Pad1.05x0.95mm_HandSolder
- R1, R2, R3, R4, R5, R7: footprint Resistor_SMD:R_0603_1608Metric -> LumiCom_Transmitter:R_0603_1608Metric
- R10, R11, R12, R9: footprint Resistor_SMD:R_0402_1005Metric_Pad0.72x0.64mm_HandSolder -> LumiCom_Transmitter:R_0402_1005Metric_Pad0.72x0.64mm_HandSolder
- R13, R14: footprint Resistor_SMD:R_1206_3216Metric_Pad1.30x1.75mm_HandSolder -> LumiCom_Transmitter:R_1206_3216Metric_Pad1.30x1.75mm_HandSolder
- R6: footprint Resistor_SMD:R_0603_1608Metric_Pad0.98x0.95mm_HandSolder -> LumiCom_Transmitter:R_0603_1608Metric_Pad0.98x0.95mm_HandSolder
