File: Transmitter/FCA/LumiCom_Transmitter.kicad_sch (KiCad schematic)
At the start: 38 parts, among them J1 V, J2 IN_B, J3 IN_A, J4 OUT_B, J5 OUT_A, U1 OPA2675

Commit message: Vendor project libraries; clean ERC/DRC on all boards
- Copy embedded footprints and symbols into each project's local library
  and repoint FPIDs / lib_ids so every project is self-contained
- Add sym-lib-table for tx_amplifier and preenfasis
- Sync footprint fields with the schematic (parity) and mark LMH34400 JP1 DNP
- Remove dangling copper arc and silkscreen overlap in LTC6268-10
- Fix LED ERC metadata errors
- All 8 boards: ERC and DRC clean (0 errors, 0 warnings)
Parts:
- C1, C2, C7: footprint Capacitor_SMD:C_0603_1608Metric_Pad1.08x0.95mm_HandSolder -> LumiCom_Transmitter:C_0603_1608Metric_Pad1.08x0.95mm_HandSolder; symbol Device:C_Small -> Lumicom_Transmitter:C_Small
- C10, C11, C3, C4, C5, C6, C8, C9: footprint Capacitor_SMD:C_0402_1005Metric_Pad0.74x0.62mm_HandSolder -> LumiCom_Transmitter:C_0402_1005Metric_Pad0.74x0.62mm_HandSolder; symbol Device:C_Small -> Lumicom_Transmitter:C_Small
- D1: symbol Device:LED -> Lumicom_Transmitter:LED
- H1, H2, H3, H4: footprint MountingHole:MountingHole_3.2mm_M3_ISO7380 -> LumiCom_Transmitter:MountingHole_3.2mm_M3_ISO7380; symbol Mechanical:MountingHole -> Lumicom_Transmitter:MountingHole
- J1: footprint TerminalBlock_Phoenix:TerminalBlock_Phoenix_MKDS-1,5-2_1x02_P5.00mm_Horizontal -> LumiCom_Transmitter:TerminalBlock_Phoenix_MKDS-1,5-2_1x02_P5.00mm_Horizontal; symbol Connector:Screw_Terminal_01x02 -> Lumicom_Transmitter:Screw_Terminal_01x02
- J2, J3, J4, J5: footprint Connector_Coaxial:SMA_Samtec_SMA-J-P-X-ST-EM1_EdgeMount -> LumiCom_Transmitter:SMA_Samtec_SMA-J-P-X-ST-EM1_EdgeMount; symbol Connector:Conn_Coaxial -> Lumicom_Transmitter:Conn_Coaxial
- JP_A0, JP_A1: footprint Connector_PinHeader_2.54mm:PinHeader_1x03_P2.54mm_Vertical -> LumiCom_Transmitter:PinHeader_1x03_P2.54mm_Vertical; symbol Jumper:Jumper_3_Bridged12 -> Lumicom_Transmitter:Jumper_3_Bridged12
- L1: footprint Inductor_SMD:L_0603_1608Metric_Pad1.05x0.95mm_HandSolder -> LumiCom_Transmitter:L_0603_1608Metric_Pad1.05x0.95mm_HandSolder; symbol Device:L_Ferrite_Small -> Lumicom_Transmitter:L_Ferrite_Small
- R1, R2, R3, R4, R5, R7: footprint Resistor_SMD:R_0603_1608Metric -> LumiCom_Transmitter:R_0603_1608Metric; symbol Device:R_Small_US -> Lumicom_Transmitter:R_Small_US
- R10, R11, R12, R9: footprint Resistor_SMD:R_0402_1005Metric_Pad0.72x0.64mm_HandSolder -> LumiCom_Transmitter:R_0402_1005Metric_Pad0.72x0.64mm_HandSolder; symbol Device:R_Small_US -> Lumicom_Transmitter:R_Small_US
- R13, R14: footprint Resistor_SMD:R_1206_3216Metric_Pad1.30x1.75mm_HandSolder -> LumiCom_Transmitter:R_1206_3216Metric_Pad1.30x1.75mm_HandSolder; symbol Device:R_Small_US -> Lumicom_Transmitter:R_Small_US
- R6: footprint Resistor_SMD:R_0603_1608Metric_Pad0.98x0.95mm_HandSolder -> LumiCom_Transmitter:R_0603_1608Metric_Pad0.98x0.95mm_HandSolder; symbol Device:R_Small_US -> Lumicom_Transmitter:R_Small_US
