File: Transmitter/LED/LED.kicad_pcb (KiCad board)
At the start: 2 copper layers, 50 x 35 mm, 11 parts, among them J1 RFPC-SMA28-F, J2 RFPC-SMA28-F, J3 Vdc

Commit message: Vendor project libraries; clean ERC/DRC on all boards
- Copy embedded footprints and symbols into each project's local library
  and repoint FPIDs / lib_ids so every project is self-contained
- Add sym-lib-table for tx_amplifier and preenfasis
- Sync footprint fields with the schematic (parity) and mark LMH34400 JP1 DNP
- Remove dangling copper arc and silkscreen overlap in LTC6268-10
- Fix LED ERC metadata errors
- All 8 boards: ERC and DRC clean (0 errors, 0 warnings)
Parts:
- C1, C2: footprint Capacitor_SMD:C_0402_1005Metric_Pad0.74x0.62mm_HandSolder -> LumiCom_Led:C_0402_1005Metric_Pad0.74x0.62mm_HandSolder
- H1, H2, H3: footprint MountingHole:MountingHole_3.2mm_M3_DIN965 -> LumiCom_Led:MountingHole_3.2mm_M3_DIN965
- J3: footprint TerminalBlock_Phoenix:TerminalBlock_Phoenix_MKDS-1,5-2_1x02_P5.00mm_Horizontal -> LumiCom_Led:TerminalBlock_Phoenix_MKDS-1,5-2_1x02_P5.00mm_Horizontal
Changed lines of the file:
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@@
 	(net 4 "Net-(J3-Pin_2)")
 	(net 5 "Net-(LED1-anode)")
-	(footprint "MountingHole:MountingHole_3.2mm_M3_DIN965"
+	(footprint "LumiCom_Led:MountingHole_3.2mm_M3_DIN965"
 		(layer "F.Cu")
 		(at 181 116)
@@
 			)
 		)
-		(property "Footprint" "MountingHole:MountingHole_3.2mm_M3_DIN965"
+		(property "Footprint" "LumiCom_Led:MountingHole_3.2mm_M3_DIN965"
 			(at 0 0 0)
 			(unlocked yes)
@@
 			)
 		)
-		(property "Description" " RF Inductors - SMD WE-CAIR Air Coil 206nH 3A AEC-Q200 "
+		(property "Description" "RF Inductors - SMD WE-CAIR Air Coil 206nH 3A AEC-Q200"
 			(at 0 0 90)
 			(unlocked yes)
@@
 		)
 	)
-	(footprint "MountingHole:MountingHole_3.2mm_M3_DIN965"
+	(footprint "LumiCom_Led:MountingHole_3.2mm_M3_DIN965"
 		(layer "F.Cu")
 		(at 181 89)
@@
 			)
 		)
-		(property "Footprint" "MountingHole:MountingHole_3.2mm_M3_DIN965"
+		(property "Footprint" "LumiCom_Led:MountingHole_3.2mm_M3_DIN965"
 			(at 0 0 0)
 			(unlocked yes)
@@
 		)
 	)
-	(footprint "MountingHole:MountingHole_3.2mm_M3_DIN965"
+	(footprint "LumiCom_Led:MountingHole_3.2mm_M3_DIN965"
 		(layer "F.Cu")
 		(at 139 116)
@@
 			)
 		)
-		(property "Footprint" "MountingHole:MountingHole_3.2mm_M3_DIN965"
+		(property "Footprint" "LumiCom_Led:MountingHole_3.2mm_M3_DIN965"
 			(at 0 0 0)
 			(unlocked yes)
@@
 		)
 	)
-	(footprint "Capacitor_SMD:C_0402_1005Metric_Pad0.74x0.62mm_HandSolder"
+	(footprint "LumiCom_Led:C_0402_1005Metric_Pad0.74x0.62mm_HandSolder"
 		(layer "F.Cu")
 		(at 150 108 90)
@@
 			)
 		)
-		(property "Footprint" "Capacitor_SMD:C_0402_1005Metric_Pad0.74x0.62mm_HandSolder"
+		(property "Footprint" "LumiCom_Led:C_0402_1005Metric_Pad0.74x0.62mm_HandSolder"
 			(at 0 0 90)
 			(unlocked yes)
@@
 		)
 	)
-	(footprint "Capacitor_SMD:C_0402_1005Metric_Pad0.74x0.62mm_HandSolder"
+	(footprint "LumiCom_Led:C_0402_1005Metric_Pad0.74x0.62mm_HandSolder"
 		(layer "F.Cu")
 		(at 170 108 90)
@@
 			)
 		)
-		(property "Footprint" "Capacitor_SMD:C_0402_1005Metric_Pad0.74x0.62mm_HandSolder"
+		(property "Footprint" "LumiCom_Led:C_0402_1005Metric_Pad0.74x0.62mm_HandSolder"
 			(at 0 0 90)
 			(unlocked yes)
@@
 		)
 	)
-	(footprint "TerminalBlock_Phoenix:TerminalBlock_Phoenix_MKDS-1,5-2_1x02_P5.00mm_Horizontal"
+	(footprint "LumiCom_Led:TerminalBlock_Phoenix_MKDS-1,5-2_1x02_P5.00mm_Horizontal"
 		(layer "B.Cu")
 		(at 141 97 90)
@@
 			)
 		)
-		(property "Footprint" "TerminalBlock_Phoenix:TerminalBlock_Phoenix_MKDS-1,5-2_1x02_P5.00mm_Horizontal"
+		(property "Footprint" "LumiCom_Led:TerminalBlock_Phoenix_MKDS-1,5-2_1x02_P5.00mm_Horizontal"
 			(at 0 0 -90)
 			(unlocked yes)
@@
 			)
 		)
-		(property "Description" " RFPC-SMA28-F GCT"
+		(property "Description" "RFPC-SMA28-F GCT"
 			(at 0 0 -90)
 			(unlocked yes)
@@
 			)
 		)
-		(property "Description" " RFPC-SMA28-F GCT"
+		(property "Description" "RFPC-SMA28-F GCT"
 			(at 0 0 -90)
 			(unlocked yes)
