File: Transmitter/LED/LED.kicad_sch (KiCad schematic)
At the start: 11 parts, among them J1 RFPC-SMA28-F, J2 RFPC-SMA28-F, J3 Vdc

Commit message: Vendor project libraries; clean ERC/DRC on all boards
- Copy embedded footprints and symbols into each project's local library
  and repoint FPIDs / lib_ids so every project is self-contained
- Add sym-lib-table for tx_amplifier and preenfasis
- Sync footprint fields with the schematic (parity) and mark LMH34400 JP1 DNP
- Remove dangling copper arc and silkscreen overlap in LTC6268-10
- Fix LED ERC metadata errors
- All 8 boards: ERC and DRC clean (0 errors, 0 warnings)
Parts:
- C1, C2: footprint Capacitor_SMD:C_0402_1005Metric_Pad0.74x0.62mm_HandSolder -> LumiCom_Led:C_0402_1005Metric_Pad0.74x0.62mm_HandSolder; symbol Device:C_Small -> LumiCom_Led:C_Small
- H1, H2, H3: footprint MountingHole:MountingHole_3.2mm_M3_DIN965 -> LumiCom_Led:MountingHole_3.2mm_M3_DIN965; symbol Mechanical:MountingHole -> LumiCom_Led:MountingHole
- J1, J2: symbol Connector:Conn_Coaxial -> LumiCom_Led:Conn_Coaxial
- J3: footprint TerminalBlock_Phoenix:TerminalBlock_Phoenix_MKDS-1,5-2_1x02_P5.00mm_Horizontal -> LumiCom_Led:TerminalBlock_Phoenix_MKDS-1,5-2_1x02_P5.00mm_Horizontal; symbol Connector:Screw_Terminal_01x02 -> LumiCom_Led:Screw_Terminal_01x02
- L1: symbol Device:L -> LumiCom_Led:L
Changed lines of the file:
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@@
+	(wire
+		(pts
+			(xy 226.06 127) (xy 231.14 127)
+		)
+		(stroke
+			(width 0)
+			(type default)
+		)
+	)
+	(symbol
+		(lib_id "LumiCom_Led:PWR_FLAG")
+		(at 231.14 127 0)
+		(unit 1)
+		(exclude_from_sim no)
+		(in_bom yes)
+		(on_board yes)
+		(dnp no)
+		(property "Reference" "#FLG01"
+			(at 231.14 125.095 0)
+			(effects
+				(font
+					(size 1.27 1.27)
+				)
+				(hide yes)
+			)
+		)
+		(property "Value" "PWR_FLAG"
+			(at 231.14 123.19 0)
+			(effects
+				(font
+					(size 1.27 1.27)
+				)
+			)
+		)
+		(property "Footprint" ""
+			(at 231.14 127 0)
+			(effects
+				(font
+					(size 1.27 1.27)
+				)
+				(hide yes)
+			)
+		)
+		(property "Datasheet" "~"
+			(at 231.14 127 0)
+			(effects
+				(font
+					(size 1.27 1.27)
+				)
+				(hide yes)
+			)
+		)
+		(property "Description" "Special symbol for telling ERC where power comes from"
+			(at 231.14 127 0)
+			(effects
+				(font
+					(size 1.27 1.27)
+				)
+				(hide yes)
+			)
+		)
+		(pin "1"
+		)
+		(instances
+			(project "LED"
+				(path "/cde9c444-d16b-47c2-b816-c8654de79d41"
+					(reference "#FLG01")
+					(unit 1)
+				)
+			)
+		)
+	)
 	(wire
 		(pts
@@
 	)
 	(symbol
-		(lib_id "Mechanical:MountingHole")
+		(lib_id "LumiCom_Led:MountingHole")
 		(at 209.55 63.5 0)
 		(unit 1)
@@
 			)
 		)
-		(property "Footprint" "MountingHole:MountingHole_3.2mm_M3_DIN965"
+		(property "Footprint" "LumiCom_Led:MountingHole_3.2mm_M3_DIN965"
 			(at 209.55 63.5 0)
 			(effects
@@
 	)
 	(symbol
-		(lib_id "Connector:Conn_Coaxial")
+		(lib_id "LumiCom_Led:Conn_Coaxial")
 		(at 177.8 119.38 0)
 		(mirror y)
@@
 	)
 	(symbol
-		(lib_id "Device:C_Small")
+		(lib_id "LumiCom_Led:C_Small")
 		(at 190.5 119.38 90)
 		(unit 1)
@@
 			)
 		)
-		(property "Footprint" "Capacitor_SMD:C_0402_1005Metric_Pad0.74x0.62mm_HandSolder"
+		(property "Footprint" "LumiCom_Led:C_0402_1005Metric_Pad0.74x0.62mm_HandSolder"
 			(at 190.5 119.38 0)
 			(effects
@@
 	)
 	(symbol
-		(lib_id "Connector:Screw_Terminal_01x02")
+		(lib_id "LumiCom_Led:Screw_Terminal_01x02")
 		(at 52.07 97.79 180)
 		(unit 1)
@@
 			)
 		)
-		(property "Footprint" "TerminalBlock_Phoenix:TerminalBlock_Phoenix_MKDS-1,5-2_1x02_P5.00mm_Horizontal"
+		(property "Footprint" "LumiCom_Led:TerminalBlock_Phoenix_MKDS-1,5-2_1x02_P5.00mm_Horizontal"
 			(at 52.07 97.79 0)
 			(effects
@@
 	)
 	(symbol
-		(lib_id "power:GND")
+		(lib_id "LumiCom_Led:GND")
 		(at 226.06 130.81 0)
 		(unit 1)
@@
 	)
 	(symbol
-		(lib_id "Mechanical:MountingHole")
+		(lib_id "LumiCom_Led:MountingHole")
 		(at 190.5 76.2 0)
 		(unit 1)
@@
 			)
 		)
-		(property "Footprint" "MountingHole:MountingHole_3.2mm_M3_DIN965"
+		(property "Footprint" "LumiCom_Led:MountingHole_3.2mm_M3_DIN965"
 			(at 190.5 76.2 0)
 			(effects
@@
 	)
 	(symbol
-		(lib_id "Device:L")
+		(lib_id "LumiCom_Led:L")
 		(at 73.66 95.25 270)
 		(unit 1)
@@
 	)
 	(symbol
-		(lib_id "power:GND")
+		(lib_id "LumiCom_Led:GND")
 		(at 177.8 124.46 0)
 		(unit 1)
@@
 	)
 	(symbol
-		(lib_id "Connector:Conn_Coaxial")
+		(lib_id "LumiCom_Led:Conn_Coaxial")
 		(at 63.5 119.38 0)
 		(mirror y)
@@
 	)
 	(symbol
-		(lib_id "Mechanical:MountingHole")
+		(lib_id "LumiCom_Led:MountingHole")
 		(at 190.5 63.5 0)
 		(unit 1)
@@
 			)
 		)
-		(property "Footprint" "MountingHole:MountingHole_3.2mm_M3_DIN965"
+		(property "Footprint" "LumiCom_Led:MountingHole_3.2mm_M3_DIN965"
 			(at 190.5 63.5 0)
 			(effects
@@
 	)
 	(symbol
-		(lib_id "power:GND")
+		(lib_id "LumiCom_Led:GND")
 		(at 111.76 130.81 0)
 		(unit 1)
@@
 	)
 	(symbol
-		(lib_id "Device:C_Small")
+		(lib_id "LumiCom_Led:C_Small")
 		(at 74.93 119.38 90)
 		(unit 1)
@@
 			)
 		)
-		(property "Footprint" "Capacitor_SMD:C_0402_1005Metric_Pad0.74x0.62mm_HandSolder"
+		(property "Footprint" "LumiCom_Led:C_0402_1005Metric_Pad0.74x0.62mm_HandSolder"
 			(at 74.93 119.38 0)
 			(effects
@@
 	)
 	(symbol
-		(lib_id "power:GND")
+		(lib_id "LumiCom_Led:GND")
 		(at 63.5 99.06 0)
 		(unit 1)
@@
 	)
 	(symbol
-		(lib_id "power:GND")
+		(lib_id "LumiCom_Led:GND")
 		(at 63.5 124.46 0)
 		(unit 1)
