File: Transmitter/PRE/filtro_T_sheet.kicad_sch (KiCad schematic)
At the start: 8 parts

Commit message: Vendor project libraries; clean ERC/DRC on all boards
- Copy embedded footprints and symbols into each project's local library
  and repoint FPIDs / lib_ids so every project is self-contained
- Add sym-lib-table for tx_amplifier and preenfasis
- Sync footprint fields with the schematic (parity) and mark LMH34400 JP1 DNP
- Remove dangling copper arc and silkscreen overlap in LTC6268-10
- Fix LED ERC metadata errors
- All 8 boards: ERC and DRC clean (0 errors, 0 warnings)
Parts:
- C3, C4: footprint Capacitor_SMD:C_0603_1608Metric_Pad1.08x0.95mm_HandSolder -> preenfasis:C_0603_1608Metric_Pad1.08x0.95mm_HandSolder; symbol Device:C -> preenfasis:C
- L3, L4: footprint Inductor_SMD:L_0603_1608Metric_Pad1.05x0.95mm_HandSolder -> preenfasis:L_0603_1608Metric_Pad1.05x0.95mm_HandSolder; symbol Device:L -> preenfasis:L
- R5, R6, R7, R8: footprint Resistor_SMD:R_0603_1608Metric_Pad0.98x0.95mm_HandSolder -> preenfasis:R_0603_1608Metric_Pad0.98x0.95mm_HandSolder; symbol Device:R_US -> preenfasis:R_US
Changed lines of the file:
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@@
 	)
 	(symbol
-		(lib_id "Device:R_US")
+		(lib_id "preenfasis:R_US")
 		(at 144.78 96.52 0)
 		(unit 1)
@@
 			)
 		)
-		(property "Footprint" "Resistor_SMD:R_0603_1608Metric_Pad0.98x0.95mm_HandSolder"
+		(property "Footprint" "preenfasis:R_0603_1608Metric_Pad0.98x0.95mm_HandSolder"
 			(at 145.796 96.774 90)
 			(effects
@@
 	)
 	(symbol
-		(lib_id "Device:L")
+		(lib_id "preenfasis:L")
 		(at 151.13 115.57 0)
 		(unit 1)
@@
 			)
 		)
-		(property "Footprint" "Inductor_SMD:L_0603_1608Metric_Pad1.05x0.95mm_HandSolder"
+		(property "Footprint" "preenfasis:L_0603_1608Metric_Pad1.05x0.95mm_HandSolder"
 			(at 151.13 115.57 0)
 			(effects
@@
 	)
 	(symbol
-		(lib_id "Device:C")
+		(lib_id "preenfasis:C")
 		(at 133.35 67.31 90)
 		(unit 1)
@@
 			)
 		)
-		(property "Footprint" "Capacitor_SMD:C_0603_1608Metric_Pad1.08x0.95mm_HandSolder"
+		(property "Footprint" "preenfasis:C_0603_1608Metric_Pad1.08x0.95mm_HandSolder"
 			(at 137.16 66.3448 0)
 			(effects
@@
 	)
 	(symbol
-		(lib_id "Device:R_US")
+		(lib_id "preenfasis:R_US")
 		(at 133.35 83.82 90)
 		(unit 1)
@@
 			)
 		)
-		(property "Footprint" "Resistor_SMD:R_0603_1608Metric_Pad0.98x0.95mm_HandSolder"
+		(property "Footprint" "preenfasis:R_0603_1608Metric_Pad0.98x0.95mm_HandSolder"
 			(at 133.604 82.804 90)
 			(effects
@@
 	)
 	(symbol
-		(lib_id "Device:C")
+		(lib_id "preenfasis:C")
 		(at 138.43 114.3 180)
 		(unit 1)
@@
 			)
 		)
-		(property "Footprint" "Capacitor_SMD:C_0603_1608Metric_Pad1.08x0.95mm_HandSolder"
+		(property "Footprint" "preenfasis:C_0603_1608Metric_Pad1.08x0.95mm_HandSolder"
 			(at 137.4648 110.49 0)
 			(effects
@@
 	)
 	(symbol
-		(lib_id "Device:R_US")
+		(lib_id "preenfasis:R_US")
 		(at 156.21 83.82 90)
 		(unit 1)
@@
 			)
 		)
-		(property "Footprint" "Resistor_SMD:R_0603_1608Metric_Pad0.98x0.95mm_HandSolder"
+		(property "Footprint" "preenfasis:R_0603_1608Metric_Pad0.98x0.95mm_HandSolder"
 			(at 156.464 82.804 90)
 			(effects
@@
 	)
 	(symbol
-		(lib_id "Device:R_US")
+		(lib_id "preenfasis:R_US")
 		(at 143.51 58.42 90)
 		(unit 1)
@@
 			)
 		)
-		(property "Footprint" "Resistor_SMD:R_0603_1608Metric_Pad0.98x0.95mm_HandSolder"
+		(property "Footprint" "preenfasis:R_0603_1608Metric_Pad0.98x0.95mm_HandSolder"
 			(at 143.764 57.404 90)
 			(effects
@@
 	)
 	(symbol
-		(lib_id "Device:L")
+		(lib_id "preenfasis:L")
 		(at 149.86 67.31 90)
 		(unit 1)
@@
 			)
 		)
-		(property "Footprint" "Inductor_SMD:L_0603_1608Metric_Pad1.05x0.95mm_HandSolder"
+		(property "Footprint" "preenfasis:L_0603_1608Metric_Pad1.05x0.95mm_HandSolder"
 			(at 149.86 67.31 0)
 			(effects
