File: Transmitter/PRE/preenfasis.kicad_sch (KiCad schematic)
At the start: 24 parts, among them J1 SMA H, J2 SMA H, J3 SMA H, J4 SMA H

Commit message: Vendor project libraries; clean ERC/DRC on all boards
- Copy embedded footprints and symbols into each project's local library
  and repoint FPIDs / lib_ids so every project is self-contained
- Add sym-lib-table for tx_amplifier and preenfasis
- Sync footprint fields with the schematic (parity) and mark LMH34400 JP1 DNP
- Remove dangling copper arc and silkscreen overlap in LTC6268-10
- Fix LED ERC metadata errors
- All 8 boards: ERC and DRC clean (0 errors, 0 warnings)
Parts:
- C1, C2, C3, C4: footprint Capacitor_SMD:C_0603_1608Metric_Pad1.08x0.95mm_HandSolder -> preenfasis:C_0603_1608Metric_Pad1.08x0.95mm_HandSolder; symbol Device:C -> preenfasis:C
- H1, H2, H3, H4: footprint MountingHole:MountingHole_3.2mm_M3_ISO7380 -> preenfasis:MountingHole_3.2mm_M3_ISO7380; symbol Mechanical:MountingHole -> preenfasis:MountingHole
- J1, J2, J3, J4: footprint Connector_Coaxial:SMA_Samtec_SMA-J-P-X-ST-EM1_EdgeMount -> preenfasis:SMA_Samtec_SMA-J-P-X-ST-EM1_EdgeMount; symbol Connector:Conn_Coaxial -> preenfasis:Conn_Coaxial
- L1, L2, L3, L4: footprint Inductor_SMD:L_0603_1608Metric_Pad1.05x0.95mm_HandSolder -> preenfasis:L_0603_1608Metric_Pad1.05x0.95mm_HandSolder; symbol Device:L -> preenfasis:L
- R1, R2, R3, R4, R5, R6, R7, R8: footprint Resistor_SMD:R_0603_1608Metric_Pad0.98x0.95mm_HandSolder -> preenfasis:R_0603_1608Metric_Pad0.98x0.95mm_HandSolder; symbol Device:R_US -> preenfasis:R_US
Changed lines of the file:
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@@
 	)
 	(symbol
-		(lib_id "Device:C")
+		(lib_id "preenfasis:C")
 		(at 87.63 121.92 180)
 		(unit 1)
@@
 			)
 		)
-		(property "Footprint" "Capacitor_SMD:C_0603_1608Metric_Pad1.08x0.95mm_HandSolder"
+		(property "Footprint" "preenfasis:C_0603_1608Metric_Pad1.08x0.95mm_HandSolder"
 			(at 86.6648 118.11 0)
 			(effects
@@
 	)
 	(symbol
-		(lib_id "Connector:Conn_Coaxial")
+		(lib_id "preenfasis:Conn_Coaxial")
 		(at 162.56 91.44 0)
 		(mirror y)
@@
 			)
 		)
-		(property "Footprint" "Connector_Coaxial:SMA_Samtec_SMA-J-P-X-ST-EM1_EdgeMount"
+		(property "Footprint" "preenfasis:SMA_Samtec_SMA-J-P-X-ST-EM1_EdgeMount"
 			(at 162.56 91.44 0)
 			(effects
@@
 	)
 	(symbol
-		(lib_id "Device:R_US")
+		(lib_id "preenfasis:R_US")
 		(at 93.98 104.14 0)
 		(unit 1)
@@
 			)
 		)
-		(property "Footprint" "Resistor_SMD:R_0603_1608Metric_Pad0.98x0.95mm_HandSolder"
+		(property "Footprint" "preenfasis:R_0603_1608Metric_Pad0.98x0.95mm_HandSolder"
 			(at 94.996 104.394 90)
 			(effects
@@
 	)
 	(symbol
-		(lib_id "Connector:Conn_Coaxial")
+		(lib_id "preenfasis:Conn_Coaxial")
 		(at 228.6 91.44 0)
 		(unit 1)
@@
 			)
 		)
-		(property "Footprint" "Connector_Coaxial:SMA_Samtec_SMA-J-P-X-ST-EM1_EdgeMount"
+		(property "Footprint" "preenfasis:SMA_Samtec_SMA-J-P-X-ST-EM1_EdgeMount"
 			(at 228.6 91.44 0)
 			(effects
@@
 	)
 	(symbol
-		(lib_id "Device:C")
+		(lib_id "preenfasis:C")
 		(at 185.42 74.93 90)
 		(unit 1)
@@
 			)
 		)
-		(property "Footprint" "Capacitor_SMD:C_0603_1608Metric_Pad1.08x0.95mm_HandSolder"
+		(property "Footprint" "preenfasis:C_0603_1608Metric_Pad1.08x0.95mm_HandSolder"
 			(at 189.23 73.9648 0)
 			(effects
@@
 	)
 	(symbol
-		(lib_id "Device:R_US")
+		(lib_id "preenfasis:R_US")
 		(at 185.42 91.44 90)
 		(unit 1)
@@
 			)
 		)
-		(property "Footprint" "Resistor_SMD:R_0603_1608Metric_Pad0.98x0.95mm_HandSolder"
+		(property "Footprint" "preenfasis:R_0603_1608Metric_Pad0.98x0.95mm_HandSolder"
 			(at 185.674 90.424 90)
 			(effects
@@
 	)
 	(symbol
-		(lib_id "Device:R_US")
+		(lib_id "preenfasis:R_US")
 		(at 208.28 91.44 90)
 		(unit 1)
@@
 			)
 		)
-		(property "Footprint" "Resistor_SMD:R_0603_1608Metric_Pad0.98x0.95mm_HandSolder"
+		(property "Footprint" "preenfasis:R_0603_1608Metric_Pad0.98x0.95mm_HandSolder"
 			(at 208.534 90.424 90)
 			(effects
@@
 	)
 	(symbol
-		(lib_id "Device:R_US")
+		(lib_id "preenfasis:R_US")
 		(at 92.71 66.04 90)
 		(unit 1)
@@
 			)
 		)
-		(property "Footprint" "Resistor_SMD:R_0603_1608Metric_Pad0.98x0.95mm_HandSolder"
+		(property "Footprint" "preenfasis:R_0603_1608Metric_Pad0.98x0.95mm_HandSolder"
 			(at 92.964 65.024 90)
 			(effects
@@
 	)
 	(symbol
-		(lib_id "Device:C")
+		(lib_id "preenfasis:C")
 		(at 82.55 74.93 90)
 		(unit 1)
@@
 			)
 		)
-		(property "Footprint" "Capacitor_SMD:C_0603_1608Metric_Pad1.08x0.95mm_HandSolder"
+		(property "Footprint" "preenfasis:C_0603_1608Metric_Pad1.08x0.95mm_HandSolder"
 			(at 86.36 73.9648 0)
 			(effects
@@
 	)
 	(symbol
-		(lib_id "Mechanical:MountingHole")
+		(lib_id "preenfasis:MountingHole")
 		(at 29.21 26.67 0)
 		(unit 1)
@@
 			)
 		)
-		(property "Footprint" "MountingHole:MountingHole_3.2mm_M3_ISO7380"
+		(property "Footprint" "preenfasis:MountingHole_3.2mm_M3_ISO7380"
 			(at 29.21 26.67 0)
 			(effects
@@
 	)
 	(symbol
-		(lib_id "Device:L")
+		(lib_id "preenfasis:L")
 		(at 99.06 74.93 90)
 		(unit 1)
@@
 			)
 		)
-		(property "Footprint" "Inductor_SMD:L_0603_1608Metric_Pad1.05x0.95mm_HandSolder"
+		(property "Footprint" "preenfasis:L_0603_1608Metric_Pad1.05x0.95mm_HandSolder"
 			(at 99.06 74.93 0)
 			(effects
@@
 	)
 	(symbol
-		(lib_id "Device:C")
+		(lib_id "preenfasis:C")
 		(at 190.5 121.92 180)
 		(unit 1)
@@
 			)
 		)
-		(property "Footprint" "Capacitor_SMD:C_0603_1608Metric_Pad1.08x0.95mm_HandSolder"
+		(property "Footprint" "preenfasis:C_0603_1608Metric_Pad1.08x0.95mm_HandSolder"
 			(at 189.5348 118.11 0)
 			(effects
@@
 	)
 	(symbol
-		(lib_id "Connector:Conn_Coaxial")
+		(lib_id "preenfasis:Conn_Coaxial")
 		(at 125.73 91.44 0)
 		(unit 1)
@@
 			)
 		)
-		(property "Footprint" "Connector_Coaxial:SMA_Samtec_SMA-J-P-X-ST-EM1_EdgeMount"
+		(property "Footprint" "preenfasis:SMA_Samtec_SMA-J-P-X-ST-EM1_EdgeMount"
 			(at 125.73 91.44 0)
 			(effects
@@
 	)
 	(symbol
-		(lib_id "Mechanical:MountingHole")
+		(lib_id "preenfasis:MountingHole")
 		(at 20.32 21.59 0)
 		(unit 1)
@@
 			)
 		)
-		(property "Footprint" "MountingHole:MountingHole_3.2mm_M3_ISO7380"
+		(property "Footprint" "preenfasis:MountingHole_3.2mm_M3_ISO7380"
 			(at 20.32 21.59 0)
 			(effects
@@
 	)
 	(symbol
-		(lib_id "Mechanical:MountingHole")
+		(lib_id "preenfasis:MountingHole")
 		(at 29.21 21.59 0)
 		(unit 1)
@@
 			)
 		)
-		(property "Footprint" "MountingHole:MountingHole_3.2mm_M3_ISO7380"
+		(property "Footprint" "preenfasis:MountingHole_3.2mm_M3_ISO7380"
 			(at 29.21 21.59 0)
 			(effects
@@
 	)
 	(symbol
-		(lib_id "Device:R_US")
+		(lib_id "preenfasis:R_US")
 		(at 195.58 66.04 90)
 		(unit 1)
@@
 			)
 		)
-		(property "Footprint" "Resistor_SMD:R_0603_1608Metric_Pad0.98x0.95mm_HandSolder"
+		(property "Footprint" "preenfasis:R_0603_1608Metric_Pad0.98x0.95mm_HandSolder"
 			(at 195.834 65.024 90)
 			(effects
@@
 	)
 	(symbol
-		(lib_id "Device:R_US")
+		(lib_id "preenfasis:R_US")
 		(at 105.41 91.44 90)
 		(unit 1)
@@
 			)
 		)
-		(property "Footprint" "Resistor_SMD:R_0603_1608Metric_Pad0.98x0.95mm_HandSolder"
+		(property "Footprint" "preenfasis:R_0603_1608Metric_Pad0.98x0.95mm_HandSolder"
 			(at 105.664 90.424 90)
 			(effects
@@
 	)
 	(symbol
-		(lib_id "Connector:Conn_Coaxial")
+		(lib_id "preenfasis:Conn_Coaxial")
 		(at 59.69 91.44 0)
 		(mirror y)
@@
 			)
 		)
-		(property "Footprint" "Connector_Coaxial:SMA_Samtec_SMA-J-P-X-ST-EM1_EdgeMount"
+		(property "Footprint" "preenfasis:SMA_Samtec_SMA-J-P-X-ST-EM1_EdgeMount"
 			(at 59.69 91.44 0)
 			(effects
@@
 	)
 	(symbol
-		(lib_id "Device:R_US")
+		(lib_id "preenfasis:R_US")
 		(at 196.85 104.14 0)
 		(unit 1)
@@
 			)
 		)
-		(property "Footprint" "Resistor_SMD:R_0603_1608Metric_Pad0.98x0.95mm_HandSolder"
+		(property "Footprint" "preenfasis:R_0603_1608Metric_Pad0.98x0.95mm_HandSolder"
 			(at 197.866 104.394 90)
 			(effects
@@
 	)
 	(symbol
-		(lib_id "Device:L")
+		(lib_id "preenfasis:L")
 		(at 203.2 123.19 0)
 		(unit 1)
@@
 			)
 		)
-		(property "Footprint" "Inductor_SMD:L_0603_1608Metric_Pad1.05x0.95mm_HandSolder"
+		(property "Footprint" "preenfasis:L_0603_1608Metric_Pad1.05x0.95mm_HandSolder"
 			(at 203.2 123.19 0)
 			(effects
@@
 	)
 	(symbol
-		(lib_id "Device:L")
+		(lib_id "preenfasis:L")
 		(at 100.33 123.19 0)
 		(unit 1)
@@
 			)
 		)
-		(property "Footprint" "Inductor_SMD:L_0603_1608Metric_Pad1.05x0.95mm_HandSolder"
+		(property "Footprint" "preenfasis:L_0603_1608Metric_Pad1.05x0.95mm_HandSolder"
 			(at 100.33 123.19 0)
 			(effects
@@
 	)
 	(symbol
-		(lib_id "Device:R_US")
+		(lib_id "preenfasis:R_US")
 		(at 82.55 91.44 90)
 		(unit 1)
@@
 			)
 		)
-		(property "Footprint" "Resistor_SMD:R_0603_1608Metric_Pad0.98x0.95mm_HandSolder"
+		(property "Footprint" "preenfasis:R_0603_1608Metric_Pad0.98x0.95mm_HandSolder"
 			(at 82.804 90.424 90)
 			(effects
@@
 	)
 	(symbol
-		(lib_id "Mechanical:MountingHole")
+		(lib_id "preenfasis:MountingHole")
 		(at 20.32 26.67 0)
 		(unit 1)
@@
 			)
 		)
-		(property "Footprint" "MountingHole:MountingHole_3.2mm_M3_ISO7380"
+		(property "Footprint" "preenfasis:MountingHole_3.2mm_M3_ISO7380"
 			(at 20.32 26.67 0)
 			(effects
@@
 	)
 	(symbol
-		(lib_id "Device:L")
+		(lib_id "preenfasis:L")
 		(at 201.93 74.93 90)
 		(unit 1)
@@
 			)
 		)
-		(property "Footprint" "Inductor_SMD:L_0603_1608Metric_Pad1.05x0.95mm_HandSolder"
+		(property "Footprint" "preenfasis:L_0603_1608Metric_Pad1.05x0.95mm_HandSolder"
 			(at 201.93 74.93 0)
 			(effects
